File: EuroMeasure-IonGaugeController.kicad_pcb (KiCad board)
At the start: 2 copper layers, 100 x 100 mm, 40 parts, among them SW1 SW_DIP_x04, SW2 RST, U1 AZ1117-3V3, U2 STM32G030CxT, Y1 16MHz

Commit message: A lot of work
Parts:
- added C1: 220uF 50V, Capacitor_SMD:CP_Elec_6.3x7.7, F.Cu at (189.4, 115.5)
- added C10: 100n, Capacitor_SMD:C_0805_2012Metric_Pad1.18x1.45mm_HandSolder, F.Cu at (-72.2, 229.8)
- added C11: 100n, Capacitor_SMD:C_0805_2012Metric_Pad1.18x1.45mm_HandSolder, F.Cu at (-69.2, 229.8)
- added C12: 100n, Capacitor_SMD:C_0805_2012Metric_Pad1.18x1.45mm_HandSolder, F.Cu at (-66.2, 229.8)
- added C13: 1n 1210, Capacitor_SMD:C_1210_3225Metric_Pad1.33x2.70mm_HandSolder, F.Cu at (-57.4, 215.6)
- added C14: 100n, Capacitor_SMD:C_0805_2012Metric_Pad1.18x1.45mm_HandSolder, F.Cu at (-63.2, 229.8)
- added C15: 3.3u 400V, Capacitor_THT:CP_Radial_D10.0mm_P3.50mm, F.Cu at (-49.4, 188.3)
- added C16: 3.3u 400V, Capacitor_THT:CP_Radial_D10.0mm_P3.50mm, F.Cu at (-37.8, 188.3)
- added C17: 10n, Capacitor_SMD:C_0805_2012Metric_Pad1.18x1.45mm_HandSolder, F.Cu at (-28.1, 206.4)
- added C2: 220uF 50V, Capacitor_SMD:CP_Elec_6.3x7.7, F.Cu at (181.2, 137.4)
- added C28: 1uF, Capacitor_SMD:C_0805_2012Metric_Pad1.18x1.45mm_HandSolder, F.Cu at (151.2, 135.1)
- added C29: 10u, Capacitor_SMD:C_0805_2012Metric_Pad1.18x1.45mm_HandSolder, B.Cu at (145.1, 138.6)
- added C3: 10u, Capacitor_SMD:C_0805_2012Metric_Pad1.18x1.45mm_HandSolder, F.Cu at (168.0, 85.4)
- added C30: C, Capacitor_SMD:C_0805_2012Metric_Pad1.18x1.45mm_HandSolder, F.Cu at (20.7, 157.9)
- added C31: 10u, Capacitor_SMD:C_0805_2012Metric_Pad1.18x1.45mm_HandSolder, B.Cu at (145.1, 142.4)
- added C32: C, Capacitor_SMD:C_0805_2012Metric_Pad1.18x1.45mm_HandSolder, F.Cu at (26.7, 157.9)
- added C33: 10u, Capacitor_SMD:C_1206_3216Metric_Pad1.33x1.80mm_HandSolder, F.Cu at (125.5, 142.4)
- added C34: 10u, Capacitor_SMD:C_1206_3216Metric_Pad1.33x1.80mm_HandSolder, F.Cu at (123.2, 142.4)
- added C35: 10u, Capacitor_SMD:C_0805_2012Metric_Pad1.18x1.45mm_HandSolder, F.Cu at (119.7, 143.8)
- added C36: 100n, Capacitor_SMD:C_0805_2012Metric_Pad1.18x1.45mm_HandSolder, F.Cu at (126.8, 128.6)
- added C37: 100n, Capacitor_SMD:C_0805_2012Metric_Pad1.18x1.45mm_HandSolder, F.Cu at (121.8, 132.3)
- added C38: 10u, Capacitor_SMD:C_1206_3216Metric_Pad1.33x1.80mm_HandSolder, F.Cu at (111.8, 142.4)
- added C39: 100n, Capacitor_SMD:C_0805_2012Metric_Pad1.18x1.45mm_HandSolder, F.Cu at (116.8, 133.1)
- added C4: 10u, Capacitor_SMD:C_0805_2012Metric_Pad1.18x1.45mm_HandSolder, F.Cu at (174.5, 87.4)
- added C40: 10n, Capacitor_SMD:C_0805_2012Metric_Pad1.18x1.45mm_HandSolder, F.Cu at (115.5, 123.9)
- added C41: 220uF 50V, Capacitor_SMD:CP_Elec_6.3x7.7, F.Cu at (154.5, 63.2)
- added C42: 330uF 25V, Capacitor_SMD:CP_Elec_10x12.5, F.Cu at (144.3, 74.9)
- added C43: 10u, Capacitor_SMD:C_0805_2012Metric_Pad1.18x1.45mm_HandSolder, F.Cu at (137.7, 72.4)
- added C44: 10u, Capacitor_SMD:C_0805_2012Metric_Pad1.18x1.45mm_HandSolder, F.Cu at (135.7, 72.4)
- added C45: 100n, Capacitor_SMD:C_0805_2012Metric_Pad1.18x1.45mm_HandSolder, F.Cu at (130.9, 81.4)
- added C46: 10n, Capacitor_SMD:C_0805_2012Metric_Pad1.18x1.45mm_HandSolder, F.Cu at (132.2, 76.4)
- added C47: 10u, Capacitor_SMD:C_0805_2012Metric_Pad1.18x1.45mm_HandSolder, F.Cu at (129.2, 64.5)
- added C48: ?, Capacitor_SMD:C_0805_2012Metric_Pad1.18x1.45mm_HandSolder, F.Cu at (125.8, 77.9)
- added C49: 100n, Capacitor_SMD:C_0805_2012Metric_Pad1.18x1.45mm_HandSolder, F.Cu at (128.8, 72.7)
- added C5: 10u, Capacitor_SMD:C_0805_2012Metric_Pad1.18x1.45mm_HandSolder, F.Cu at (171.8, 85.4)
- added C50: 100n, Capacitor_SMD:C_0805_2012Metric_Pad1.18x1.45mm_HandSolder, F.Cu at (128.8, 68.3)
- added C51: ?, Capacitor_SMD:C_0805_2012Metric_Pad1.18x1.45mm_HandSolder, F.Cu at (125.8, 63.1)
- added C52: 330uF 25V, Capacitor_SMD:CP_Elec_10x12.5, F.Cu at (144.3, 61.5)
- added C53: 100n, Capacitor_SMD:C_0805_2012Metric_Pad1.18x1.45mm_HandSolder, F.Cu at (133.5, 61.1)
- added C54: 10u, Capacitor_SMD:C_0805_2012Metric_Pad1.18x1.45mm_HandSolder, F.Cu at (135.7, 68.6)
- added C55: 100p, Capacitor_SMD:C_0805_2012Metric_Pad1.18x1.45mm_HandSolder, F.Cu at (129.5, 60.7)
- added C56: 100n, Capacitor_SMD:C_0805_2012Metric_Pad1.18x1.45mm_HandSolder, F.Cu at (131.5, 61.0)
- added C57: 10u, Capacitor_SMD:C_0805_2012Metric_Pad1.18x1.45mm_HandSolder, F.Cu at (137.7, 68.6)
- added C6: 100n, Capacitor_SMD:C_0805_2012Metric_Pad1.18x1.45mm_HandSolder, F.Cu at (175.3, 82.5)
- added C7: 10u, Capacitor_SMD:C_0805_2012Metric_Pad1.18x1.45mm_HandSolder, F.Cu at (-30.5, 197.3)
- added C8: 10u, Capacitor_SMD:C_0805_2012Metric_Pad1.18x1.45mm_HandSolder, F.Cu at (-30.5, 200.3)
- added C9: 220n, Capacitor_THT:C_Disc_D6.0mm_W2.5mm_P5.00mm, F.Cu at (149.6, 101.7)
- added D1: 1N4148, Diode_SMD:D_SOD-323F, F.Cu at (-27.9, 229.1)
- added D10: MURS160BJ, Diode_SMD:D_SOD-123F, F.Cu at (129.8, 141.6)
- added D11: MURS160BJ, Diode_SMD:D_SOD-123F, F.Cu at (129.8, 139.3)
- added D12: 1N4148, Diode_SMD:D_SOD-323F, F.Cu at (118.7, 137.4)
- added D13: 1N4148, Diode_SMD:D_SOD-323F, F.Cu at (120.8, 140.9)
- added D2: MURS160BJ, Diode_SMD:D_SMB, F.Cu at (116.2, 105.0)
- added D3: MURS160BJ, Diode_SMD:D_SMB, F.Cu at (116.2, 100.5)
- added D4: MURS160BJ, Diode_SMD:D_SMB, F.Cu at (116.2, 95.9)
- added D5: MURS160BJ, Diode_SMD:D_SMB, F.Cu at (116.2, 91.3)
- added D8: D_PMEG200G20ELRX, Diode_SMD:D_SOD-123F, F.Cu at (129.8, 143.9)
- added D9: MURS160BJ, Diode_SMD:D_SOD-123F, F.Cu at (129.8, 137.0)
- added DZ1: 14V, Package_TO_SOT_SMD:SOT-23-3, F.Cu at (-49.1, 229.2)
- added DZ2: 2V4, Package_TO_SOT_SMD:SOT-363_SC-70-6_Handsoldering, F.Cu at (-53.2, 229.6)
- added DZ3: 2V4, Package_TO_SOT_SMD:SOT-363_SC-70-6_Handsoldering, F.Cu at (119.5, 122.0)
- added F1: Polyfuse 2A, MEMS_Passive:Fuse_Littlefuse_3425L, F.Cu at (181.8, 114.8)
- added F3: Polyfuse 2A, MEMS_Passive:Fuse_Littlefuse_3425L, F.Cu at (165.0, 62.9)
- added FL1: ~, MEMS_Passive:T_FL2015, F.Cu at (145.3, 104.3)
- added HS1: Heatsink 274-3AB, MEMS_Custom:274-3AB, F.Cu at (124.8, 140.4)
- added J1: Conn_01x04, Connector_Dsub:DSUB-9_Female_Horizontal_P2.77x2.54mm_EdgePinOffset9.40mm, F.Cu at (370.0, 49.4)
- added K1: UD2-5NU, MEMS_Passive:Relay_DPDT_Kemet_UC2_NU, F.Cu at (174.2, 117.7)
- added L1: 220u, Inductor_SMD:L_12x12mm_H8mm, F.Cu at (184.4, 127.1)
- added L2: 220u, Inductor_SMD:L_12x12mm_H8mm, F.Cu at (155.7, 114.1)
- added L4: 220u, Inductor_SMD:L_1210_3225Metric_Pad1.42x2.65mm_HandSolder, F.Cu at (124.3, 138.2)
- added L5: 220u, Inductor_SMD:L_12x12mm_H8mm, F.Cu at (156.6, 74.0)
- added L6: 8.2u, MEMS_Passive:L_Bourns_SRP7030, F.Cu at (123.5, 70.5)
- added Q1: FZT1053A, Package_TO_SOT_SMD:SOT-223-3_TabPin2, F.Cu at (155.8, 102.8)
- added Q2: IRF540SPBF, Package_TO_SOT_SMD:TO-263-2, F.Cu at (159.9, 127.0)
- added Q3: FZT1053A, Package_TO_SOT_SMD:SOT-223-3_TabPin2, F.Cu at (155.8, 95.3)
- added R1: 1, Resistor_SMD:R_0805_2012Metric_Pad1.20x1.40mm_HandSolder, F.Cu at (168.9, 82.5)
- added R10: 30k, Resistor_SMD:R_0805_2012Metric_Pad1.20x1.40mm_HandSolder, F.Cu at (-41.9, 206.6)
- added R11: 100R 0.1% 5PPM, Resistor_SMD:R_0805_2012Metric_Pad1.20x1.40mm_HandSolder, F.Cu at (-38.9, 206.6)
- added R12: 100R 0.1% 5PPM, Resistor_SMD:R_0805_2012Metric_Pad1.20x1.40mm_HandSolder, F.Cu at (-36.0, 206.6)
- added R13: 1k, Resistor_SMD:R_0805_2012Metric, F.Cu at (-45.4, 228.9)
- added R2: 10, Resistor_SMD:R_0805_2012Metric_Pad1.20x1.40mm_HandSolder, F.Cu at (170.9, 82.5)
- added R20: 1.5k, Resistor_SMD:R_0805_2012Metric_Pad1.20x1.40mm_HandSolder, F.Cu at (154.0, 145.0)
- added R21: 22k, Resistor_SMD:R_0805_2012Metric_Pad1.20x1.40mm_HandSolder, F.Cu at (153.2, 135.1)
- added R22: 50k, Resistor_SMD:R_0805_2012Metric_Pad1.20x1.40mm_HandSolder, F.Cu at (149.2, 135.1)
- added R23: 21k, Resistor_SMD:R_0805_2012Metric_Pad1.20x1.40mm_HandSolder, F.Cu at (152.6, 140.8)
- added R24: 2.2k, Resistor_SMD:R_0805_2012Metric_Pad1.20x1.40mm_HandSolder, F.Cu at (150.2, 145.0)
- added R25: R, Resistor_SMD:R_0805_2012Metric_Pad1.20x1.40mm_HandSolder, F.Cu at (16.5, 171.9)
- added R26: R, Resistor_SMD:R_0805_2012Metric_Pad1.20x1.40mm_HandSolder, F.Cu at (19.5, 171.9)
- added R27: 4.7k, Resistor_SMD:R_0805_2012Metric_Pad1.20x1.40mm_HandSolder, F.Cu at (119.7, 145.8)
- added R28: 240R, Resistor_SMD:R_0805_2012Metric_Pad1.20x1.40mm_HandSolder, F.Cu at (118.8, 140.9)
- added R29: 1k 0.1% 5PPM, Resistor_SMD:R_0805_2012Metric_Pad1.20x1.40mm_HandSolder, F.Cu at (114.8, 133.1)
- added R3: 10k, Resistor_SMD:R_0805_2012Metric_Pad1.20x1.40mm_HandSolder, F.Cu at (-53.7, 206.6)
- added R30: 1k 0.1% 5PPM, Resistor_SMD:R_0805_2012Metric_Pad1.20x1.40mm_HandSolder, F.Cu at (115.3, 127.8)
- added R31: 10k 0.1% 5PPM, Resistor_SMD:R_0805_2012Metric_Pad1.20x1.40mm_HandSolder, F.Cu at (117.2, 127.8)
- added R32: 1k, Resistor_SMD:R_0805_2012Metric, F.Cu at (118.2, 124.8)
- added R33: 10k, Resistor_SMD:R_0805_2012Metric_Pad1.20x1.40mm_HandSolder, F.Cu at (134.6, 79.4)
- added R34: 1k, Resistor_SMD:R_0805_2012Metric_Pad1.20x1.40mm_HandSolder, F.Cu at (130.9, 79.4)
- added R35: 47k, Resistor_SMD:R_0805_2012Metric_Pad1.20x1.40mm_HandSolder, F.Cu at (134.2, 76.4)
- added R36: ?, Resistor_SMD:R_0805_2012Metric_Pad1.20x1.40mm_HandSolder, F.Cu at (125.8, 75.9)
- added R37: ?, Resistor_SMD:R_0805_2012Metric_Pad1.20x1.40mm_HandSolder, F.Cu at (125.8, 65.1)
- added R38: 20m 1%, Resistor_SMD:R_2010_5025Metric_Pad1.40x2.65mm_HandSolder, F.Cu at (136.1, 63.2)
- added R39: 8.2k, Resistor_SMD:R_0805_2012Metric_Pad1.20x1.40mm_HandSolder, F.Cu at (131.5, 64.8)
- added R40: 0R, Resistor_SMD:R_0805_2012Metric_Pad1.20x1.40mm_HandSolder, F.Cu at (133.5, 64.8)
- added R41: 100k, Resistor_SMD:R_0805_2012Metric_Pad1.20x1.40mm_HandSolder, F.Cu at (132.8, 57.8)
- added R42: 8.2k, Resistor_SMD:R_0805_2012Metric_Pad1.20x1.40mm_HandSolder, F.Cu at (129.0, 57.8)
- added R43: 10k, Resistor_SMD:R_0805_2012Metric_Pad1.20x1.40mm_HandSolder, F.Cu at (132.8, 55.8)
- added R44: 1k, Resistor_SMD:R_0805_2012Metric_Pad1.20x1.40mm_HandSolder, F.Cu at (129.0, 55.8)
- added R45: R_1210_820Ohm, Resistor_SMD:R_1210_3225Metric_Pad1.30x2.65mm_HandSolder, F.Cu at (144.8, 108.8)
- added R5: 1k, Resistor_SMD:R_0805_2012Metric_Pad1.20x1.40mm_HandSolder, F.Cu at (-50.7, 206.6)
- added R6: 470k, Resistor_SMD:R_0805_2012Metric_Pad1.20x1.40mm_HandSolder, F.Cu at (-47.8, 206.6)
- added R7: 1k 0.5W, Resistor_SMD:R_1210_3225Metric_Pad1.30x2.65mm_HandSolder, F.Cu at (-57.4, 221.6)
- added R8: 10k, Resistor_SMD:R_0805_2012Metric_Pad1.20x1.40mm_HandSolder, F.Cu at (-44.8, 206.6)
- added R9: 2M, Resistor_THT:R_Axial_DIN0204_L3.6mm_D1.6mm_P7.62mm_Horizontal, F.Cu at (-31.0, 220.3)
- added TP1: Cathode_I, MEMS_Custom:TestPoint_Pad_D1.0mm, F.Cu at (161.2, 83.4)
- added TP2: Grid_I, MEMS_Custom:TestPoint_Pad_D1.0mm, F.Cu at (161.2, 86.4)
- added TP3: Anode_I, MEMS_Custom:TestPoint_Pad_D1.0mm, F.Cu at (161.2, 89.5)
- added TP4: Cathode_V, MEMS_Custom:TestPoint_Pad_D1.0mm, F.Cu at (161.2, 92.5)
- added TP5: ADC_DRDY, MEMS_Custom:TestPoint_Pad_D1.0mm, F.Cu at (-55.4, 114.8)
- added TP6: ADC_RESET, MEMS_Custom:TestPoint_Pad_D1.0mm, F.Cu at (-55.4, 117.9)
- added TP7: ADC_CS, MEMS_Custom:TestPoint_Pad_D1.0mm, F.Cu at (-55.4, 120.9)
- added U1: ADS131M04-WQFN, Package_DFN_QFN:WQFN-20-1EP_3x3mm_P0.4mm_EP1.7x1.7mm, F.Cu at (170.1, 88.6)
- added U10: TPS55289, MEMS_IC:TPS55289, F.Cu at (131.9, 70.5)
- added U2: TL072, Package_SO:SO-8_3.9x4.9mm_P1.27mm, F.Cu at (-28.8, 188.2)
- added U3: 3.0V, Package_TO_SOT_SMD:SOT-23, F.Cu at (-32.0, 206.4)
- added U6: SN6507, MEMS_IC:SN6507, F.Cu at (149.8, 140.5)
- added U7: T_750316856, MEMS_Passive:750316856, F.Cu at (140.3, 140.5)
- added U8: LM317HVT_TO-220-3, Package_TO_SOT_THT:TO-220-3_Horizontal_TabUp, F.Cu at (114.5, 143.0)
- added U9: OPA2187, Package_SO:SOIC-8_3.9x4.9mm_P1.27mm, F.Cu at (122.0, 128.6)
- added X1: 8.192MHz, Oscillator:Oscillator_SMD_ECS_2520MV-xxx-xx-4Pin_2.5x2.0mm, F.Cu at (175.4, 85.0)
- renumbered C1 to C18, C2 to C19, C3 to C20, C4 to C21, C5 to C22, C6 to C23, C7 to C24, C8 to C25, C9 to C26, C10 to C27, D1 to D6, D2 to D7, F1 to F2, L1 to L3, R1 to R14, R2 to R15, R3 to R16, R4 to R17, R5 to R18, R6 to R19, TP3 to TP10, TP4 to TP11, TP5 to TP12, TP6 to TP13, TP7 to TP14, TP8 to TP15, TP9 to TP16, TP10 to TP17, TP1 to TP8, TP2 to TP9, U1 to U4, U2 to U5
Connections:
- net /EuroMeasure/SPI1_MISO renamed /DOUT
- net /EuroMeasure/SPI1_MOSI renamed /DIN
- net /EuroMeasure/SPI1_SCK renamed /SCLK
- U5 pad 28: /EuroMeasure/PA8 -> /DRDY
- U5 pad 29: /EuroMeasure/PA9 -> /RESET
- U5 pad 32: /EuroMeasure/PA10 -> /CS
Routing:
- net GND: track 36.6 -> 88.2 mm, vias 18 -> 41
- net /Anode: track 0.00 -> 23.9 mm
- net /Cathode: track 0.00 -> 18.7 mm, vias 0 -> 2
- net Net-(U10-VIN): track 0.00 -> 15.5 mm
- net /Grid Supply/heatsink_2: track 0.00 -> 15.2 mm
- net /Grid Supply/heatsink_1: track 0.00 -> 15.2 mm
- net Net-(U10-ISP): track 0.00 -> 14.7 mm
- net Net-(D12-A): track 0.00 -> 13.8 mm
- net Net-(D8-K): track 0.00 -> 13.8 mm
- net Net-(Q3-B): track 0.00 -> 13.1 mm, vias 0 -> 2
- net Net-(U10-SW1): track 0.00 -> 12.6 mm
- net Net-(U10-SW2): track 0.00 -> 12.6 mm
- net Net-(U10-EN/UVLO): track 0.00 -> 11.0 mm
- net Net-(R40-Pad2): track 0.00 -> 9.84 mm, vias 0 -> 2
- net Net-(Q1-B): track 0.00 -> 8.81 mm
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
Commit message: Copper layout done
Parts:
- added C58: 200p C0G, Capacitor_SMD:C_0805_2012Metric_Pad1.18x1.45mm_HandSolder, F.Cu at (121.9, 124.7)
- added R4: 1k, Resistor_SMD:R_0805_2012Metric_Pad1.20x1.40mm_HandSolder, F.Cu at (157.0, 84.8)
- added R46: 1k, Resistor_SMD:R_0805_2012Metric_Pad1.20x1.40mm_HandSolder, F.Cu at (153.3, 85.3)
- C7, C8: moved to B.Cu
- J1: value Conn_01x04 -> Conn_02x05_Odd_Even; footprint Connector_Dsub:DSUB-9_Female_Horizontal_P2.77x2.54mm_EdgePinOffset9.40mm -> Connector_IDC:IDC-Header_2x05_P2.54mm_Vertical
- moved J1 266.1 mm to (106.2, 84.3), turned to 180 degrees
- moved DZ2 259.9 mm to (157.3, 77.0)
- moved R13 254.0 mm to (160.9, 80.7), turned to 180 degrees
- moved C11 246.8 mm to (145.2, 107.7)
- moved C10 243.1 mm to (140.6, 112.3), turned to 180 degrees
- moved C12 240.7 mm to (139.4, 104.7), turned to 0 degrees
- moved R11 238.8 mm to (162.1, 77.7), turned to 90 degrees
- moved R12 237.0 mm to (161.0, 74.8), turned to 180 degrees
- moved TP5 232.2 mm to (175.6, 90.0)
- moved C14 231.5 mm to (134.8, 109.9), turned to 0 degrees
- moved TP7 230.7 mm to (173.7, 93.2)
- moved TP6 230.5 mm to (173.6, 91.0)
- moved C17 227.8 mm to (159.9, 77.7), turned to 90 degrees
- moved D1 222.4 mm to (167.6, 123.2), turned to 180 degrees
- moved DZ1 222.0 mm to (134.6, 104.5), turned to 180 degrees
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Connections:
- net Net-(C41-Pad1) renamed /Cathode Supply/15V_Filtered
- net Net-(C7-Pad2) renamed /Grid Supply/5V_Lockouted
- net Net-(U10-SW1) renamed /Cathode Supply/SW1
- C17 pad 1: /AIN0N -> /AIN2N
- C40 pad 1: /AIN1N -> /AIN3N
- DZ2 pad 6: /AIN0N -> /AIN2N
- DZ3 pad 6: /AIN1N -> /AIN3N
- J1 pad 1: /Grid -> unconnected-(J1-Pin_1-Pad1)
- J1 pad 3: /Cathode -> /Grid
- J1 pad 4: GND -> unconnected-(J1-Pin_4-Pad4)
- J1 pad 5: (no net) -> unconnected-(J1-Pin_5-Pad5)
- J1 pad 6: (no net) -> unconnected-(J1-Pin_6-Pad6)
- J1 pad 7: (no net) -> /Cathode
- J1 pad 8: (no net) -> /Cathode
- J1 pad 9: (no net) -> GND
- R13 pad 2: /AIN0N -> /AIN2N
- R31 pad 2: /AIN1N -> /AIN3N
- R32 pad 2: /AIN1N -> /AIN3N
- R43 pad 2: /AIN3N -> /AIN0N
- R44 pad 1: /AIN3N -> /AIN0N
- U10 pad 16: /AIN2N -> /AIN1N
Routing:
- net 5V_INPUT: track 100.0 -> 256.4 mm, vias 1 -> 15
- net 15V_INPUT: track 5.26 -> 142.7 mm, vias 0 -> 15
- net -15V_INPUT: track 4.91 -> 136.2 mm, vias 0 -> 3
- net /AIN3N: track 1.80 -> 113.1 mm, vias 0 -> 3
- net GNDD: track 0.00 -> 97.8 mm, vias 0 -> 2
- net /AIN0N: track 0.00 -> 73.8 mm
- net /AIN1N: track 7.17 -> 80.2 mm, vias 0 -> 2
- net +5VL: track 6.79 -> 74.8 mm, vias 0 -> 22
- net /Anode: track 23.9 -> 89.9 mm
- net /EuroMeasure/SCL_INT: track 29.2 -> 94.7 mm, vias 3 -> 6
- net /EuroMeasure/SDA_INT: track 29.4 -> 93.5 mm, vias 3 -> 6
- net +3.3V: track 94.7 -> 136.1 mm, vias 5 -> 7
- net /Grid: track 0.00 -> 38.0 mm
- net /Grid Supply/5V_Lockouted: track 0.00 -> 38.0 mm, vias 0 -> 20
- net Net-(D2-K): track 0.00 -> 36.8 mm
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- added copper zone on B.Cu, net +5VL
- added copper zone on F.Cu, net +5VL
- added copper zone on B.Cu, net /Cathode
- added copper zone on F.Cu, net /Cathode
- added copper zone on F.Cu, net /Cathode Supply/15V_Filtered
- added copper zone on F.Cu, net /Cathode Supply/SW1
- added copper zone on B.Cu, net /Grid Supply/5V_Lockouted
- added copper zone on F.Cu, net /Grid Supply/5V_Lockouted
- added copper zone on F.Cu, net /Grid Supply/heatsink_1
- added copper zone on F.Cu, net /Grid Supply/heatsink_2
- added copper zone on F.Cu, net /Grid Supply/heatsink_3
- added copper zone on B.Cu, net Net-(Q1-E)
- added copper zone on F.Cu, net Net-(Q1-E)
- added copper zone on B.Cu, net Net-(U10-ISP)
- added copper zone on F.Cu, net Net-(U10-ISP)
- added copper zone on F.Cu, net Net-(U10-SW2)
- added copper zone on B.Cu, net Net-(U10-VIN)
- added copper zone on F.Cu, net Net-(U10-VIN)

Commit message: Clean DRC
Routing:
- net 5V_INPUT: track 256.4 -> 254.4 mm

Commit message: Final 1.0.0 version
Other:
- board text added: "JLCJLCJLC"
Changed lines of the file:
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@@
       (layer "F.SilkS" (type "Top Silk Screen"))
       (layer "F.Paste" (type "Top Solder Paste"))
-      (layer "F.Mask" (type "Top Solder Mask") (thickness 0.01))
+      (layer "F.Mask" (type "Top Solder Mask") (color "Red") (thickness 0.01))
       (layer "F.Cu" (type "copper") (thickness 0.035))
       (layer "dielectric 1" (type "core") (thickness 1.51) (material "FR4") (epsilon_r 4.5) (loss_tangent 0.02))
       (layer "B.Cu" (type "copper") (thickness 0.035))
-      (layer "B.Mask" (type "Bottom Solder Mask") (thickness 0.01))
+      (layer "B.Mask" (type "Bottom Solder Mask") (color "Red") (thickness 0.01))
       (layer "B.Paste" (type "Bottom Solder Paste"))
       (layer "B.SilkS" (type "Bottom Silk Screen"))
-      (copper_finish "None")
+      (copper_finish "HAL SnPb")
       (dielectric_constraints no)
     )
@@
     (property "ki_keywords" "Adjustable Voltage Regulator 1.5A Positive")
     (attr through_hole)
-    (fp_text reference "U8" (at -2.545 -0.625 90) (layer "F.SilkS")
+    (fp_text reference "U8" (at 2.54 20.58 90) (layer "F.SilkS")
         (effects (font (size 1 1) (thickness 0.15)))
     )
@@
   (footprint "MEMS_Passive:750316856" (layer "F.Cu")
     (at 140.35 140.5 180)
-    (property "MPN:" "750316856")
-    (property "Mouser:" "710-750316856")
+    (property "MPN" "750316856")
+    (property "Mouser" "710-750316856")
     (property "Sheetfile" "anode_supply.kicad_sch")
     (property "Sheetname" "Anode Supply")
@@
   (footprint "MEMS_IC:SN6507" (layer "F.Cu")
     (at 149.85 140.5 90)
+    (property "MPN" "SN6507DGQR")
+    (property "Mouser" "595-SN6507DGQR")
     (property "Sheetfile" "anode_supply.kicad_sch")
     (property "Sheetname" "Anode Supply")
@@
     (descr "Through hole IDC box header, 2x05, 2.54mm pitch, DIN 41651 / IEC 60603-13, double rows, https://docs.google.com/spreadsheets/d/16SsEcesNF15N3Lb4niX7dcUr-NY5_MFPQhobNuNppn4/edit#gid=0")
     (tags "Through hole vertical IDC box header THT 2x05 2.54mm double row")
+    (property "MPN" "NO_MPN")
     (property "Sheetfile" "EuroMeasure-IonGaugeController.kicad_sch")
     (property "Sheetname" "")
@@
     (descr "SO, 8 Pin (https://www.nxp.com/docs/en/data-sheet/PCF8523.pdf), generated with kicad-footprint-generator ipc_gullwing_generator.py")
     (tags "SO SO")
+    (property "MPN" "TL082IDRQ1")
     (property "Mouser" "595-TL082IDRQ1")
     (property "Sheetfile" "grid_supply.kicad_sch")
@@
   (gr_rect (start 100 50) (end 200 150)
     (stroke (width 0.1) (type default)) (fill none) (layer "Edge.Cuts"))
+  (gr_text "JLCJLCJLC" (at 127 88.4) (layer "F.SilkS")
+    (effects (font (size 1 1) (thickness 0.15)) (justify left bottom))
+  )
   (segment (start 169.0375 85.4) (end 169.0375 83.6375) (width 0.2) (layer "F.Cu") (net 1))
   (segment (start 169.7 86.0625) (end 169.0375 85.4) (width 0.2) (layer "F.Cu") (net 1))
