File: EuroMeasure-IonGaugeController.kicad_pcb (KiCad board)
At the start: 2 copper layers, 100 x 100 mm, 172 parts, among them J1 Conn_02x05_Odd_Even, K1 UD2-5NU, Q1 FZT1053A, Q2 IRF540SPBF, Q3 FZT1053A, SW1 SW_DIP_x04, SW2 RST, U1 ADS131M04-WQFN, U10 TPS55289, U2 TL072, U3 3.0V, U4 AZ1117-3V3, U5 STM32G030CxT, U6 SN6507, U7 T_750316856, U8 LM317HVT_TO-220-3, U9 OPA2187, X1 8.192MHz, Y1 16MHz

Commit message: Revision 1.1.0. DRC clean
Parts:
- added R47: 0R, Resistor_SMD:R_0805_2012Metric_Pad1.20x1.40mm_HandSolder, F.Cu at (124.7, 76.5)
- C13: value 1n 1210 -> 1n X7R
- C40: value 10n -> 200p C0G
- C58: value 200p C0G -> 10n
- J1: value Conn_02x05_Odd_Even -> Gauge Connector; footprint Connector_IDC:IDC-Header_2x05_P2.54mm_Vertical -> Connector_IDC:IDC-Header_2x05_P2.54mm_Horizontal
- TP1: value Cathode_I -> Grid_I
- TP10: value SPI1_MOSI -> MOSI
- TP2: value Grid_I -> Anode_I
- TP3: value Anode_I -> Cathode_I
- TP5: value ADC_DRDY -> DRDY
- TP6: value ADC_RESET -> RESET
- TP7: value ADC_CS -> CS
- TP8: value SPI1_SCK -> SCK
- TP9: value SPI1_MISO -> MISO
- moved TP15 42.8 mm to (190.9, 101.8)
- moved TP14 21.9 mm to (171.1, 92.8)
- moved TP16 21.0 mm to (174.8, 62.2)
- moved TP13 12.4 mm to (178.4, 82.9)
- moved C10 6.51 mm to (145.2, 107.7), turned to 90 degrees
- moved C11 6.47 mm to (140.7, 112.3), turned to 0 degrees
- moved C58 6.45 mm to (115.5, 123.9), turned to -90 degrees
- moved C40 6.41 mm to (121.8, 124.7), turned to 180 degrees
- moved TP2 5.39 mm to (169.1, 92.2)
- moved TP4 5.39 mm to (166.7, 87.4)
- moved U4 0.14 mm to (182.9, 71.9)
- moved L1 0.14 mm to (184.5, 127.0)
- moved C6 0.10 mm to (175.4, 82.2)
- moved R13 0.07 mm to (160.8, 80.7)
- moved C1 0.07 mm to (189.5, 115.5)
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Connections:
- net +5VL renamed /Anode Supply/5V_IN
- net /AIN1N renamed /ADC/2
- net /AIN2N renamed /ADC/3
- net /Anode renamed /ANODE
- net /CLK renamed /ADC/CLK
- net /CS renamed /ADC/CS
- net /Cathode renamed /CATHODE
- net /Cathode Supply/15V_Filtered renamed Net-(C41-Pad1)
- net /DIN renamed /ADC/DIN
- net /DOUT renamed /ADC/DOUT
- net /DRDY renamed /ADC/DRDY
- net /EuroMeasure/ADR0 renamed /MCU/ADR0
- net /EuroMeasure/ADR1 renamed /MCU/ADR1
- net /EuroMeasure/ADR2 renamed /MCU/ADR2
- net /EuroMeasure/ADR3 renamed /MCU/ADR3
- net /EuroMeasure/GP0 renamed /Backplane connector/GP0
- net /EuroMeasure/GP1 renamed /Backplane connector/GP1
- net /EuroMeasure/LED renamed /MCU/LED
- net /EuroMeasure/MCU_PWR renamed /MCU/3V3_MCU
- net /EuroMeasure/OSC32_IN renamed /MCU/OSC32_IN
- net /EuroMeasure/OSC32_OUT renamed /MCU/OSC32_OUT
- net /EuroMeasure/OSC_IN renamed /MCU/OSC_IN
- net /EuroMeasure/OSC_OUT renamed /MCU/OSC_OUT
- net /EuroMeasure/RDY renamed /Backplane connector/RDY
- net /EuroMeasure/RGB_LED renamed /MCU/RGB_LED
- net /EuroMeasure/RST renamed /Backplane connector/RST
- net /EuroMeasure/RST_LOCAL renamed /Backplane connector/RST_LOCAL
- net /EuroMeasure/RX_DEBUG renamed /Backplane connector/RX
- net /EuroMeasure/SCL_EXT renamed /Backplane connector/SCL
- net /EuroMeasure/SCL_INT renamed /Cathode Supply/SCL
- net /EuroMeasure/SDA_EXT renamed /Backplane connector/SDA
- net /EuroMeasure/SDA_INT renamed /Cathode Supply/SDA
- net /EuroMeasure/SWCLK renamed /Backplane connector/SWCLK
- net /EuroMeasure/SWDIO renamed /Backplane connector/SWDIO
- net /EuroMeasure/TRG renamed /Backplane connector/TRG
- net /EuroMeasure/TX_DEBUG renamed /Backplane connector/TX
- net /Grid renamed /GRID
- net /RESET renamed /ADC/RESET
- net /SCLK renamed /ADC/SCLK
- net 5V_INPUT renamed +5V
- net Net-(D12-A) renamed /Anode Current Measurement/IN
- net Net-(D2-A) renamed /Grid Supply/GRID_AC0
- net Net-(D2-K) renamed /Grid Supply/GRID_Unfiltered
- net Net-(D4-K) renamed /Grid Supply/GRID_AC1
- net Net-(U10-VIN) renamed /Cathode Supply/15V_FILTERED
- net Net-(U4-VI) renamed /PSU/5V_FUSED
- B1 pad 1: -15V_INPUT -> -15V
- B1 pad 10: 15V_INPUT -> +15V
- B1 pad 15: /EuroMeasure/~{LOCKOUT} -> /Backplane connector/~{LOCKOUT}
- B1 pad 2: -15V_INPUT -> -15V
- B1 pad 28: /EuroMeasure/NC4 -> unconnected-(B1A-NC4-Pad28)
- B1 pad 29: /EuroMeasure/NC5 -> unconnected-(B1A-NC5-Pad29)
- B1 pad 30: /EuroMeasure/NC6 -> unconnected-(B1A-NC6-Pad30)
- B1 pad 9: 15V_INPUT -> +15V
- B1 pad D1: /EuroMeasure/RGB_OUT -> unconnected-(B1B-DO-PadD1)
- C10 pad 2: 15V_INPUT -> +15V
- C11 pad 1: -15V_INPUT -> -15V
- C14 pad 1: GND -> GNDD
- C36 pad 1: 15V_INPUT -> +15V
- C37 pad 2: -15V_INPUT -> -15V
- C40 pad 1: /AIN3N -> Net-(U9A--)
- C40 pad 2: GND -> Net-(C40-Pad2)
- C58 pad 1: Net-(U9A--) -> /ADC/4
- C58 pad 2: Net-(C58-Pad2) -> GND
- D1 pad 1: ~{LOCKOUT} -> /Backplane connector/~{LOCKOUT}
- DZ3 pad 6: /AIN3N -> /ADC/4
- F3 pad 2: 15V_INPUT -> +15V
- K1 pad 1: ~{LOCKOUT} -> /Backplane connector/~{LOCKOUT}
- L2 pad 1: Net-(Q1-E) -> /Grid Supply/heatsink_3
- L2 pad 2: /Grid Supply/heatsink_3 -> /Grid Supply/heatsink_4
- Q1 pad 3: Net-(Q1-E) -> /Grid Supply/heatsink_3
- Q2 pad 2: /Grid Supply/heatsink_3 -> /Grid Supply/heatsink_4
- Q3 pad 3: Net-(Q1-E) -> /Grid Supply/heatsink_3
- R31 pad 2: /AIN3N -> /ADC/4
- R32 pad 1: Net-(C58-Pad2) -> Net-(C40-Pad2)
- R32 pad 2: /AIN3N -> /ADC/4
- R43 pad 2: /AIN0N -> /ADC/1
- R44 pad 1: /AIN0N -> /ADC/1
- TP2 pad 1: /AIN0N -> /ADC/4
- TP4 pad 1: /AIN3N -> /ADC/1
- U1 pad 2: /AIN0N -> /ADC/1
- U1 pad 7: /AIN3N -> /ADC/4
- U2 pad 4: 15V_INPUT -> -15V
- U2 pad 8: -15V_INPUT -> +15V
- U3 pad 2: GND -> GNDD
- U5 pad 1: /EuroMeasure/PC13 -> unconnected-(U5-PC13-Pad1)
- U5 pad 12: /EuroMeasure/PA1 -> unconnected-(U5-PA1-Pad12)
- U5 pad 15: /EuroMeasure/PA4 -> unconnected-(U5-PA4-Pad15)
- U5 pad 19: /EuroMeasure/PB0 -> unconnected-(U5-PB0-Pad19)
- U5 pad 20: /EuroMeasure/PB1 -> unconnected-(U5-PB1-Pad20)
- U5 pad 21: /EuroMeasure/PB2 -> unconnected-(U5-PB2-Pad21)
- U5 pad 22: /EuroMeasure/~{LOCKOUT} -> /Backplane connector/~{LOCKOUT}
- U5 pad 25: /EuroMeasure/SPI2_SCK -> unconnected-(U5-PB13-Pad25)
- U5 pad 26: /EuroMeasure/SPI2_MISO -> unconnected-(U5-PB14-Pad26)
- U5 pad 27: /EuroMeasure/SPI2_MOSI -> unconnected-(U5-PB15-Pad27)
- U5 pad 30: /EuroMeasure/PC6 -> unconnected-(U5-PC6-Pad30)
- U5 pad 37: /EuroMeasure/PA15 -> unconnected-(U5-PA15-Pad37)
- U5 pad 42: /EuroMeasure/PB3 -> unconnected-(U5-PB3-Pad42)
- U5 pad 43: /EuroMeasure/PB4 -> unconnected-(U5-PB4-Pad43)
- U5 pad 44: /EuroMeasure/PB5 -> unconnected-(U5-PB5-Pad44)
- U9 pad 1: Net-(C58-Pad2) -> Net-(C40-Pad2)
- U9 pad 4: -15V_INPUT -> -15V
- U9 pad 8: 15V_INPUT -> +15V
Routing:
- net +15V: track 0.00 -> 144.2 mm, vias 0 -> 16
- net 15V_INPUT: track 142.7 -> 0.00 mm, vias 15 -> 0
- net -15V_INPUT: track 136.2 -> 0.00 mm, vias 3 -> 0
- net -15V: track 0.00 -> 130.4 mm, vias 0 -> 3
- net /ADC/4: track 0.00 -> 113.1 mm, vias 0 -> 3
- net /AIN3N: track 113.1 -> 0.00 mm, vias 3 -> 0
- net /Backplane connector/~{LOCKOUT}: track 0.00 -> 100.3 mm, vias 0 -> 5
- net /ADC/1: track 0.00 -> 73.8 mm
- net /AIN0N: track 73.8 -> 0.00 mm
- net /EuroMeasure/~{LOCKOUT}: track 30.9 -> 0.00 mm, vias 1 -> 0
- net GNDD: track 97.8 -> 105.2 mm, vias 2 -> 3
- net ~{LOCKOUT}: track 5.14 -> 0.00 mm
- net Net-(C58-Pad2): track 3.76 -> 0.00 mm
- net Net-(C40-Pad2): track 0.00 -> 3.76 mm
- net GND: vias 239 -> 244
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- added copper zone on B.Cu, net /Grid Supply/heatsink_3
- added copper zone on F.Cu, net /Grid Supply/heatsink_4
- removed copper zone on B.Cu, net Net-(Q1-E)
- removed copper zone on F.Cu, net Net-(Q1-E)

Commit message: Everything clear. Gerbers generated
Parts:
- C19: renamed from C30; value C -> ~
- C21: renamed from C32; value C -> ~
- C33: renamed from C48; value ? -> ~
- C36: renamed from C51; value ? -> ~
- FL1: value ~ -> FL2015-4L
- R20: renamed from R25; value R -> ~
- R21: renamed from R26; value R -> ~
- R30: renamed from R36; value ? -> ~
- R31: renamed from R37; value ? -> ~
- renumbered C22 to C1, C11 to C10, C9 to C11, C13 to C12, C12 to C13, C28 to C17, C29 to C18, C23 to C2, C31 to C20, C33 to C22, C34 to C23, C35 to C24, C38 to C25, C41 to C26, C42 to C27, C43 to C28, C44 to C29, C24 to C3, C45 to C30, C46 to C31, C47 to C32, C49 to C34, C50 to C35, C52 to C37, C53 to C38, C54 to C39, C25 to C4, C55 to C40, C56 to C41, C57 to C42, C3 to C43, C4 to C44, C5 to C45, C6 to C46, C39 to C47, C36 to C48, C37 to C49, C26 to C5, C40 to C50, C58 to C51, C17 to C52, C18 to C53, C19 to C54, C1 to C55, C2 to C56, C20 to C57, C21 to C58, C27 to C6, C10 to C9, D6 to D1, D7 to D2, D1 to D3, D2 to D4, D3 to D5, D4 to D6, D5 to D7, DZ3 to DZ2, DZ2 to DZ3, F3 to F1, F1 to F3, L3 to L1, L4 to L3, L5 to L4, L6 to L5, L1 to L6, R16 to R1, R6 to R10, R7 to R11, R8 to R12, R9 to R13, R10 to R14, R20 to R15, R21 to R16, R22 to R17, R23 to R18, R24 to R19, R17 to R2, R27 to R22, R28 to R23, R4 to R24, R46 to R25, R47 to R26, R33 to R27, R34 to R28, R35 to R29, R18 to R3, R38 to R32, R39 to R33, R40 to R34, R41 to R35, R42 to R36, R43 to R37, R44 to R38, R1 to R39, R19 to R4, R2 to R40, R29 to R41, R30 to R42, R31 to R43, R32 to R44, R11 to R45, R12 to R46, R13 to R47, R14 to R5, R15 to R6, R3 to R7, R45 to R8, R5 to R9, SW2 to SW1, SW1 to SW2, TP4 to TP1, TP9 to TP10, TP10 to TP11, TP5 to TP12, TP6 to TP13, TP7 to TP14, TP11 to TP15, TP12 to TP16, TP3 to TP2, TP2 to TP3, TP1 to TP4, TP13 to TP5, TP14 to TP6, TP15 to TP7, TP16 to TP8, TP8 to TP9, U5 to U1, U4 to U10, U6 to U4, U7 to U5, U8 to U6, U10 to U7, U1 to U8
