File: MCU.kicad_sch (KiCad schematic)
At the start: 36 parts, among them SW1 SW_DIP_x04, SW2 RST, U5 STM32G030CxT, Y1 16MHz

Commit message: Everything clear. Gerbers generated
Parts:
- C2: renamed from C23; DNP DNP -> (none)
- C3: renamed from C24; DNP DNP -> (none)
- TP10: renamed from TP9; symbol Connector:TestPoint -> MEMS_Other:TP_1mm_via; now left out of the parts list
- TP11: renamed from TP10; symbol Connector:TestPoint -> MEMS_Other:TP_1mm_via; now left out of the parts list
- TP12: renamed from TP5; symbol Connector:TestPoint -> MEMS_Other:TP_1mm_via; now left out of the parts list
- TP13: renamed from TP6; symbol Connector:TestPoint -> MEMS_Other:TP_1mm_via; now left out of the parts list
- TP14: renamed from TP7; symbol Connector:TestPoint -> MEMS_Other:TP_1mm_via; now left out of the parts list
- TP15: renamed from TP11; symbol Connector:TestPoint -> MEMS_Other:TP_1mm_via; now left out of the parts list
- TP16: renamed from TP12; symbol Connector:TestPoint -> MEMS_Other:TP_1mm_via; now left out of the parts list
- TP5: renamed from TP13; symbol Connector:TestPoint -> MEMS_Other:TP_1mm_via; now left out of the parts list
- TP6: renamed from TP14; symbol Connector:TestPoint -> MEMS_Other:TP_1mm_via; now left out of the parts list
- TP7: renamed from TP15; symbol Connector:TestPoint -> MEMS_Other:TP_1mm_via; now left out of the parts list
- TP8: renamed from TP16; symbol Connector:TestPoint -> MEMS_Other:TP_1mm_via; now left out of the parts list
- TP9: renamed from TP8; symbol Connector:TestPoint -> MEMS_Other:TP_1mm_via; now left out of the parts list
- renumbered C22 to C1, C25 to C4, C26 to C5, C27 to C6, D6 to D1, D7 to D2, L3 to L1, R16 to R1, R17 to R2, R18 to R3, R19 to R4, R14 to R5, R15 to R6, SW2 to SW1, SW1 to SW2, U5 to U1
