File: adc.kicad_sch (KiCad schematic)
At the start: 8 parts, among them U1 ADS131M04-WQFN, X1 8.192MHz

Commit message: Everything clear. Gerbers generated
Parts:
- renumbered C3 to C43, C4 to C44, C5 to C45, C6 to C46, R1 to R39, R2 to R40, U1 to U8
Changed lines of the file:
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@@
   (symbol (lib_id "Device:R_Small") (at 134.62 49.53 180) (unit 1)
     (in_bom yes) (on_board yes) (dnp no) (fields_autoplaced)
-    (property "Reference" "R1" (at 136.525 48.2599 0)
+    (property "Reference" "R39" (at 136.525 48.2599 0)
       (effects (font (size 1.27 1.27)) (justify right))
     )
@@
       (project "EuroMeasure-IonGaugeController"
         (path "/9c84a828-ebcc-4f88-b5cc-11be4f5044ad/8647b0da-fa27-42a5-91f6-9b9bb070f7f7"
-          (reference "R1") (unit 1)
+          (reference "R39") (unit 1)
         )
       )
@@
   (symbol (lib_id "power:GND") (at 124.46 57.15 0) (unit 1)
     (in_bom yes) (on_board yes) (dnp no) (fields_autoplaced)
-    (property "Reference" "#PWR07" (at 124.46 63.5 0)
+    (property "Reference" "#PWR072" (at 124.46 63.5 0)
       (effects (font (size 1.27 1.27)) hide)
     )
@@
       (project "EuroMeasure-IonGaugeController"
         (path "/9c84a828-ebcc-4f88-b5cc-11be4f5044ad/8647b0da-fa27-42a5-91f6-9b9bb070f7f7"
-          (reference "#PWR07") (unit 1)
+          (reference "#PWR072") (unit 1)
         )
       )
@@
   (symbol (lib_id "power:GND") (at 134.62 109.22 0) (unit 1)
     (in_bom yes) (on_board yes) (dnp no) (fields_autoplaced)
-    (property "Reference" "#PWR09" (at 134.62 115.57 0)
+    (property "Reference" "#PWR073" (at 134.62 115.57 0)
       (effects (font (size 1.27 1.27)) hide)
     )
@@
       (project "EuroMeasure-IonGaugeController"
         (path "/9c84a828-ebcc-4f88-b5cc-11be4f5044ad/8647b0da-fa27-42a5-91f6-9b9bb070f7f7"
-          (reference "#PWR09") (unit 1)
+          (reference "#PWR073") (unit 1)
         )
       )
@@
   (symbol (lib_id "power:GND") (at 147.32 107.95 0) (unit 1)
     (in_bom yes) (on_board yes) (dnp no) (fields_autoplaced)
-    (property "Reference" "#PWR012" (at 147.32 114.3 0)
+    (property "Reference" "#PWR075" (at 147.32 114.3 0)
       (effects (font (size 1.27 1.27)) hide)
     )
@@
       (project "EuroMeasure-IonGaugeController"
         (path "/9c84a828-ebcc-4f88-b5cc-11be4f5044ad/8647b0da-fa27-42a5-91f6-9b9bb070f7f7"
-          (reference "#PWR012") (unit 1)
+          (reference "#PWR075") (unit 1)
         )
       )
@@
   (symbol (lib_id "Device:C_Small") (at 153.67 55.88 90) (unit 1)
     (in_bom yes) (on_board yes) (dnp no) (fields_autoplaced)
-    (property "Reference" "C5" (at 153.6763 49.53 90)
+    (property "Reference" "C45" (at 153.6763 49.53 90)
       (effects (font (size 1.27 1.27)))
     )
@@
       (project "EuroMeasure-IonGaugeController"
         (path "/9c84a828-ebcc-4f88-b5cc-11be4f5044ad/8647b0da-fa27-42a5-91f6-9b9bb070f7f7"
-          (reference "C5") (unit 1)
+          (reference "C45") (unit 1)
         )
       )
@@
   (symbol (lib_id "power:GND") (at 198.12 88.9 0) (unit 1)
     (in_bom yes) (on_board yes) (dnp no) (fields_autoplaced)
-    (property "Reference" "#PWR016" (at 198.12 95.25 0)
+    (property "Reference" "#PWR078" (at 198.12 95.25 0)
       (effects (font (size 1.27 1.27)) hide)
     )
@@
       (project "EuroMeasure-IonGaugeController"
         (path "/9c84a828-ebcc-4f88-b5cc-11be4f5044ad/8647b0da-fa27-42a5-91f6-9b9bb070f7f7"
-          (reference "#PWR016") (unit 1)
+          (reference "#PWR078") (unit 1)
         )
       )
@@
   (symbol (lib_id "power:GND") (at 142.24 116.84 0) (unit 1)
     (in_bom yes) (on_board yes) (dnp no) (fields_autoplaced)
-    (property "Reference" "#PWR010" (at 142.24 123.19 0)
+    (property "Reference" "#PWR074" (at 142.24 123.19 0)
       (effects (font (size 1.27 1.27)) hide)
     )
@@
       (project "EuroMeasure-IonGaugeController"
         (path "/9c84a828-ebcc-4f88-b5cc-11be4f5044ad/8647b0da-fa27-42a5-91f6-9b9bb070f7f7"
-          (reference "#PWR010") (unit 1)
+          (reference "#PWR074") (unit 1)
         )
       )
@@
   (symbol (lib_id "power:GND") (at 157.48 57.15 0) (unit 1)
     (in_bom yes) (on_board yes) (dnp no) (fields_autoplaced)
-    (property "Reference" "#PWR013" (at 157.48 63.5 0)
+    (property "Reference" "#PWR076" (at 157.48 63.5 0)
       (effects (font (size 1.27 1.27)) hide)
     )
@@
       (project "EuroMeasure-IonGaugeController"
         (path "/9c84a828-ebcc-4f88-b5cc-11be4f5044ad/8647b0da-fa27-42a5-91f6-9b9bb070f7f7"
-          (reference "#PWR013") (unit 1)
+          (reference "#PWR076") (unit 1)
         )
       )
@@
   (symbol (lib_id "power:GND") (at 121.92 99.06 0) (unit 1)
     (in_bom yes) (on_board yes) (dnp no) (fields_autoplaced)
-    (property "Reference" "#PWR06" (at 121.92 105.41 0)
+    (property "Reference" "#PWR071" (at 121.92 105.41 0)
       (effects (font (size 1.27 1.27)) hide)
     )
@@
       (project "EuroMeasure-IonGaugeController"
         (path "/9c84a828-ebcc-4f88-b5cc-11be4f5044ad/8647b0da-fa27-42a5-91f6-9b9bb070f7f7"
-          (reference "#PWR06") (unit 1)
+          (reference "#PWR071") (unit 1)
         )
       )
@@
   (symbol (lib_id "power:PWR_FLAG") (at 134.62 53.34 270) (unit 1)
     (in_bom yes) (on_board yes) (dnp no) (fields_autoplaced)
-    (property "Reference" "#FLG01" (at 136.525 53.34 0)
+    (property "Reference" "#FLG04" (at 136.525 53.34 0)
       (effects (font (size 1.27 1.27)) hide)
     )
@@
       (project "EuroMeasure-IonGaugeController"
         (path "/9c84a828-ebcc-4f88-b5cc-11be4f5044ad/8647b0da-fa27-42a5-91f6-9b9bb070f7f7"
-          (reference "#FLG01") (unit 1)
+          (reference "#FLG04") (unit 1)
         )
       )
@@
   (symbol (lib_id "power:PWR_FLAG") (at 147.32 53.34 90) (unit 1)
     (in_bom yes) (on_board yes) (dnp no) (fields_autoplaced)
-    (property "Reference" "#FLG02" (at 145.415 53.34 0)
+    (property "Reference" "#FLG05" (at 145.415 53.34 0)
       (effects (font (size 1.27 1.27)) hide)
     )
@@
       (project "EuroMeasure-IonGaugeController"
         (path "/9c84a828-ebcc-4f88-b5cc-11be4f5044ad/8647b0da-fa27-42a5-91f6-9b9bb070f7f7"
-          (reference "#FLG02") (unit 1)
+          (reference "#FLG05") (unit 1)
         )
       )
@@
   (symbol (lib_id "Device:C_Small") (at 142.24 113.03 0) (unit 1)
     (in_bom yes) (on_board yes) (dnp no)
-    (property "Reference" "C4" (at 144.78 114.3 0)
+    (property "Reference" "C44" (at 144.78 114.3 0)
       (effects (font (size 1.27 1.27)) (justify left))
     )
@@
       (project "EuroMeasure-IonGaugeController"
         (path "/9c84a828-ebcc-4f88-b5cc-11be4f5044ad/8647b0da-fa27-42a5-91f6-9b9bb070f7f7"
-          (reference "C4") (unit 1)
+          (reference "C44") (unit 1)
         )
       )
@@
   (symbol (lib_id "Device:C_Small") (at 198.12 85.09 0) (mirror x) (unit 1)
     (in_bom yes) (on_board yes) (dnp no) (fields_autoplaced)
-    (property "Reference" "C6" (at 200.66 83.8136 0)
+    (property "Reference" "C46" (at 200.66 83.8136 0)
       (effects (font (size 1.27 1.27)) (justify left))
     )
@@
       (project "EuroMeasure-IonGaugeController"
         (path "/9c84a828-ebcc-4f88-b5cc-11be4f5044ad/8647b0da-fa27-42a5-91f6-9b9bb070f7f7"
-          (reference "C6") (unit 1)
+          (reference "C46") (unit 1)
         )
       )
@@
   (symbol (lib_id "power:GND") (at 182.88 99.06 0) (unit 1)
     (in_bom yes) (on_board yes) (dnp no) (fields_autoplaced)
-    (property "Reference" "#PWR015" (at 182.88 105.41 0)
+    (property "Reference" "#PWR077" (at 182.88 105.41 0)
       (effects (font (size 1.27 1.27)) hide)
     )
@@
       (project "EuroMeasure-IonGaugeController"
         (path "/9c84a828-ebcc-4f88-b5cc-11be4f5044ad/8647b0da-fa27-42a5-91f6-9b9bb070f7f7"
-          (reference "#PWR015") (unit 1)
+          (reference "#PWR077") (unit 1)
         )
       )
@@
   (symbol (lib_id "Device:C_Small") (at 128.27 55.88 90) (unit 1)
     (in_bom yes) (on_board yes) (dnp no)
-    (property "Reference" "C3" (at 129.54 49.53 90)
+    (property "Reference" "C43" (at 129.54 49.53 90)
       (effects (font (size 1.27 1.27)) (justify left))
     )
@@
       (project "EuroMeasure-IonGaugeController"
         (path "/9c84a828-ebcc-4f88-b5cc-11be4f5044ad/8647b0da-fa27-42a5-91f6-9b9bb070f7f7"
-          (reference "C3") (unit 1)
+          (reference "C43") (unit 1)
         )
       )
@@
   (symbol (lib_id "Device:R_Small") (at 147.32 49.53 180) (unit 1)
     (in_bom yes) (on_board yes) (dnp no)
-    (property "Reference" "R2" (at 142.24 48.26 0)
+    (property "Reference" "R40" (at 142.24 48.26 0)
       (effects (font (size 1.27 1.27)) (justify right))
     )
@@
       (project "EuroMeasure-IonGaugeController"
         (path "/9c84a828-ebcc-4f88-b5cc-11be4f5044ad/8647b0da-fa27-42a5-91f6-9b9bb070f7f7"
-          (reference "R2") (unit 1)
+          (reference "R40") (unit 1)
         )
       )
@@
   (symbol (lib_id "MEMS_IC:ADS131M04-WQFN") (at 154.94 68.58 0) (unit 1)
     (in_bom yes) (on_board yes) (dnp no)
-    (property "Reference" "U1" (at 138.43 62.23 0)
+    (property "Reference" "U8" (at 138.43 62.23 0)
       (effects (font (size 1.27 1.27)) (justify left))
     )
@@
       (project "EuroMeasure-IonGaugeController"
         (path "/9c84a828-ebcc-4f88-b5cc-11be4f5044ad/8647b0da-fa27-42a5-91f6-9b9bb070f7f7"
-          (reference "U1") (unit 1)
-        )
-      )
+          (reference "U8") (unit 1)
+        )
+      )
