File: anode_current_measurement.kicad_sch (KiCad schematic)
At the start: 9 parts, among them U9 OPA2187

Commit message: Everything clear. Gerbers generated
Parts:
- added C48, C49: 100n, Capacitor_SMD:C_0805_2012Metric_Pad1.18x1.45mm_HandSolder, symbol Device:C_Small
- added unit 3 of U9
- added unit 2 of U9
- renumbered C39 to C47, C40 to C50, C58 to C51, DZ3 to DZ2, R29 to R41, R30 to R42, R31 to R43, R32 to R44
Connections:
- net GND: now also C48.2, C49.1, U9.5 (+)
- net In renamed IN
- net Out renamed OUT
- new net: U9.6 (-), U9.7
- new net +15V: C48.1, U9.8 (V+)
- new net -15V: C49.2, U9.4 (V-)
Other:
- note added: "Unused OP-amp"
- title: (none) -> EuroMeasure Ion Gauge Controller
