File: anode_supply.kicad_sch (KiCad schematic)
At the start: 30 parts, among them T1 Transformer_SP_1S, U1 SN6507, U6 LM317_SOT-223

Commit message: A lot of work
Parts:
- removed C14, C7: 220uF 50V, Capacitor_SMD:CP_Elec_6.3x7.7, symbol MEMS_Passive:C_Elec-220uf-50V
- removed D12: 6V3, Diode_SMD:D_MELF, symbol MEMS_Discrete-semiconductor:D_Zener_6V3_TZMB3V6-GS08
- removed D7, D8: MURS160BJ, Diode_SMD:D_SMB, symbol MEMS_Discrete-semiconductor:D_MURS160-13-F
- removed L2: 100u, MEMS_Passive:L_Bourns_PM2110, symbol MEMS_Passive:L_100u_choke
- removed L5: L, symbol Device:L
- removed R15: 200R, symbol Device:R_Small
- removed T1: Transformer_SP_1S, symbol Device:Transformer_SP_1S
- removed unit 2 of U1
- removed U6: LM317_SOT-223, Package_TO_SOT_SMD:SOT-223-3_TabPin2, symbol MEMS_IC:LM317_SOT223
- added C29: 10u, Capacitor_SMD:C_0805_2012Metric_Pad1.18x1.45mm_HandSolder, symbol Device:C_Small
- added C38: 10u, Capacitor_SMD:C_1206_3216Metric_Pad1.33x1.80mm_HandSolder, symbol Device:C_Small
- added C9 (x3): 100n, Capacitor_SMD:C_0805_2012Metric_Pad1.18x1.45mm_HandSolder, symbol Device:C_Small
- added D12, D13: 1N4148, Diode_SMD:D_SOD-323F, symbol MEMS_Discrete-semiconductor:D_1N4148WS-SOD323
- added D9 (x2): MURS160BJ, Diode_SMD:D_SOD-123F, symbol MEMS_Discrete-semiconductor:D_PMEG200G20ELRX
- added DZ3: 2V4, Package_TO_SOT_SMD:SOT-363_SC-70-6_Handsoldering, symbol MEMS_Discrete-semiconductor:D_Zener_2V4_dual_MMBZ5221BS
- added HS1: Heatsink 274-3AB, MEMS_Custom:274-3AB, symbol MEMS_Electromechanical:Heatsink
- added L4: 220u, Inductor_SMD:L_1210_3225Metric_Pad1.42x2.65mm_HandSolder, symbol MEMS_Passive:L_1210_220u
- added R2: 2.2k, Resistor_SMD:R_0805_2012Metric_Pad1.20x1.40mm_HandSolder, symbol Device:R_Small
- added R29, R30: 1k 0.1% 5PPM, Resistor_SMD:R_0805_2012Metric_Pad1.20x1.40mm_HandSolder, symbol MEMS_Passive:R_0805_1k_0.1%_5PPM
- added R31: 10k 0.1% 5PPM, Resistor_SMD:R_0805_2012Metric_Pad1.20x1.40mm_HandSolder, symbol MEMS_Passive:R_0805_10k_0.1%_5PPM
- added U7: T_750316856, MEMS_Passive:750316856, symbol MEMS_Passive:T_750316856
- added U8: LM317HVT_TO-220-3, Package_TO_SOT_THT:TO-220-3_Horizontal_TabUp, symbol MEMS_IC:LM317HVT_TO-220-3
- added U9: OPA2187, Package_SO:SOIC-8_3.9x4.9mm_P1.27mm, symbol MEMS_IC:OPA2187IDR-SOIC8
- C1: value C -> 1uF
- C31: renamed from C30; footprint (none) -> Capacitor_SMD:C_0805_2012Metric_Pad1.18x1.45mm_HandSolder
- C33, C34: footprint (none) -> Capacitor_SMD:C_1206_3216Metric_Pad1.33x1.80mm_HandSolder; MPN (none) -> GRM32EC72A106KE05L; Mouser (none) -> 81-GRM32EC72A106KE05
- C35: footprint (none) -> Capacitor_SMD:C_0805_2012Metric_Pad1.18x1.45mm_HandSolder
- C9: value 100n -> 10n; footprint Capacitor_SMD:C_0805_2012Metric -> Capacitor_SMD:C_0805_2012Metric_Pad1.18x1.45mm_HandSolder; now fitted
- D6: value MURS160BJ -> D_PMEG200G20ELRX; footprint Diode_SMD:D_SMB -> Diode_SMD:D_SOD-123F; symbol MEMS_Discrete-semiconductor:D_MURS160-13-F -> MEMS_Discrete-semiconductor:D_PMEG200G20ELRX; MPN MURS160-13-F -> PMEG200G20ELRX; Mouser 621-MURS160-F -> 771-PMEG200G20ELRX
- D9: footprint Diode_SMD:D_SMB -> Diode_SMD:D_SOD-123F; symbol MEMS_Discrete-semiconductor:D_MURS160-13-F -> MEMS_Discrete-semiconductor:D_PMEG200G20ELRX; MPN MURS160-13-F -> PMEG200G20ELRX; Mouser 621-MURS160-F -> 771-PMEG200G20ELRX
- R2: value R -> 1.5k
- R27: renamed from R25; footprint (none) -> Resistor_SMD:R_0805_2012Metric_Pad1.20x1.40mm_HandSolder
- R28: renamed from R26; footprint (none) -> Resistor_SMD:R_0805_2012Metric_Pad1.20x1.40mm_HandSolder
- R3: value R -> 22k
- R4: value R -> 50k
- R5: value R -> 21k; now not fitted
Connections:
- net +15V: now also C9.1, U9.8 (V+)
- net GND: now also C9.2, C29.1, C9.1, C9.2, C9.2, DZ3.3 (K), R29.2, R30.2, U9.5 (+)
- net I_Monitor: now also C9.1, DZ3.6 (K), R31.2
- net SW1: now also U7.1
- net SW2: now also U7.3
- net at R27.1, R28.2: now also C35.2, D13.2 (A), U8.1 (ADJ)
- net at C34.2: now also D12.1 (K), L4.2, U8.3 (VI)
- net +5VL: now reaches C31.2, U1.3 (VCC)
- net +5VL: now also C29.2, R2.2, U7.2
- net at R2.2, U1.4 (EN/UVLO): now also R2.1
- net at D9.1 (K): now also D9.2 (A), U7.4; no longer D6.2 (A)
- net at C33.2, D6.1 (K): now also D9.1 (K), L4.1
- net at R28.1: now also C38.2, C9.1, D12.2 (A), D13.1 (K), R29.1, U8.2 (VO), U9.3 (+); no longer C35.2
- net at R16.1: now also U9.1
- net -25V_Grid_Supply renamed -25V_Anode_Supply
- net -25V_Anode_Supply: now also C38.1, D9.2 (A)
- new net: D6.2 (A), D9.1 (K), U7.6
- new net: DZ3.1 (A), DZ3.4 (A)
- new net: R30.1, R31.1, U9.2 (-)
- new net: U9.6 (-), U9.7
- new net -15V: C9.2, U9.4 (V-)
- no-connect marks 1 -> 2
Other:
- note added: "0.1V/100uA"
- note added: "1.1V/100uA"
- note added: "1:4.67 Min freq V-T: 5V / 15Vus = 333kHz Supported frequencies: 200-600kHz"
- note added: "Current Limit: 50k - 500mA"
- note added: "DC-DC Output current: 0.5A/2/4.67=54mA Output voltage: 46.7V"
- note added: "EN Voltage: 1.5V*(1+2.2k/1.5k) = 3.8V"
- note added: "Heavily derated, only about 2.5uF each"
- note added: "Operating frequency: ~500kHz"
- note added: "Output Voltage: 1.25V*(1+4.7k/240) +4.7kOhm*50uA = 26V"
- note added: "Populate to decrease emissions"
- note added: "Snubber circuits to decrease emissions"
- note added: "Soft-Start Time: 1uF / (275uA - 0.6V/50k) = 3.8ms"
- note added: "~-75dB at working frequency, per simulation"
- moved on the sheet: C1, C31, C33, C4, C6, D6, D9, R16, R2, R27, R28, R3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

Commit message: Copper layout done
Parts:
- added C9: 200p C0G, Capacitor_SMD:C_0805_2012Metric_Pad1.18x1.45mm_HandSolder, symbol Device:C_Small
Connections:
- net at R16.1, U9.1: now also C9.2
- net at R30.1, R31.1, U9.2 (-): now also C9.1
Other:
- moved on the sheet: C9, DZ3A, DZ3B, R16, R30, R31

Commit message: Final 1.0.0 version
Parts:
- U1: MPN (none) -> SN6507DGQR; Mouser (none) -> 595-SN6507DGQR
- U7: MPN (none) -> 750316856; MPN: 750316856 -> (none); Mouser (none) -> 710-750316856; Mouser: 710-750316856 -> (none)
Changed lines of the file:
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@@
+      (effects (font (size 1.27 1.27)) hide)
+    )
+    (property "MPN" "SN6507DGQR" (at 116.84 130.81 0)
+      (effects (font (size 1.27 1.27)) hide)
+    )
+    (property "Mouser" "595-SN6507DGQR" (at 116.84 128.27 0)
       (effects (font (size 1.27 1.27)) hide)
     )
@@
       (effects (font (size 1.27 1.27)) hide)
     )
-    (property "MPN:" "750316856" (at 163.83 170.18 0)
-      (effects (font (size 1.27 1.27)) hide)
-    )
-    (property "Mouser:" "710-750316856" (at 163.83 172.72 0)
+    (property "MPN" "750316856" (at 163.83 170.18 0)
+      (effects (font (size 1.27 1.27)) hide)
+    )
+    (property "Mouser" "710-750316856" (at 163.83 172.72 0)
       (effects (font (size 1.27 1.27)) hide)
     )
@@
       (effects (font (size 1.27 1.27)) hide)
     )
-    (property "Datasheet" "https://www.murata.com/en-global/products/productdetail?partno=GRM32EC72A106KE05%23" (at 195.58 151.13 0)
+    (property "Datasheet" "~" (at 195.58 151.13 0)
       (effects (font (size 1.27 1.27)) hide)
     )
@@
       (effects (font (size 1.27 1.27)) hide)
     )
-    (property "Datasheet" "https://www.murata.com/en-global/products/productdetail?partno=GRM32EC72A106KE05%23" (at 257.81 151.13 0)
+    (property "Datasheet" "~" (at 257.81 151.13 0)
       (effects (font (size 1.27 1.27)) hide)
     )
@@
       (effects (font (size 1.27 1.27)) hide)
     )
-    (property "Datasheet" "https://www.murata.com/en-global/products/productdetail?partno=GRM32EC72A106KE05%23" (at 208.28 151.13 0)
-      (effects (font (size 1.27 1.27)) hide)
-    )
+    (property "Datasheet" "~" (at 208.28 151.13 0)
+      (effects (font (size 1.27 1.27)) hide)
+    )

Commit message: Revision 1.1.0. DRC clean
Parts:
- removed C9 (x3): 100n, Capacitor_SMD:C_0805_2012Metric_Pad1.18x1.45mm_HandSolder, symbol Device:C_Small
- removed C9: 200p C0G, Capacitor_SMD:C_0805_2012Metric_Pad1.18x1.45mm_HandSolder, symbol Device:C_Small
- removed C9: 10n, Capacitor_SMD:C_0805_2012Metric_Pad1.18x1.45mm_HandSolder, symbol Device:C_Small
- removed DZ3: 2V4, Package_TO_SOT_SMD:SOT-363_SC-70-6_Handsoldering, symbol MEMS_Discrete-semiconductor:D_Zener_2V4_dual_MMBZ5221BS
- removed R16: 1k, Resistor_SMD:R_0805_2012Metric, symbol Device:R_Small
- removed R29, R30: 1k 0.1% 5PPM, Resistor_SMD:R_0805_2012Metric_Pad1.20x1.40mm_HandSolder, symbol MEMS_Passive:R_0805_1k_0.1%_5PPM
- removed R31: 10k 0.1% 5PPM, Resistor_SMD:R_0805_2012Metric_Pad1.20x1.40mm_HandSolder, symbol MEMS_Passive:R_0805_10k_0.1%_5PPM
- removed U9: OPA2187, Package_SO:SOIC-8_3.9x4.9mm_P1.27mm, symbol MEMS_IC:OPA2187IDR-SOIC8
Connections:
- net +: now reaches C38.2, D12.2 (A), D13.1 (K), R28.1, U8.2 (VO)
- net +5VL renamed 5V_IN
- net -25V_Anode_Supply renamed -
Other:
- note removed: "0.1V/100uA"
- note removed: "1.1V/100uA"

Commit message: Everything clear. Gerbers generated
Parts:
- C4, C6: value C -> ~
- R6, R7: value R -> ~
- renumbered C29 to C18, C31 to C20, C33 to C22, C34 to C23, C35 to C24, C38 to C25, L4 to L3, R27 to R22, R28 to R23, U7 to U5, U8 to U6
Other:
- moved on the sheet: C1, C18, C20, C22, C23, C24, C25, C4, C6, D12, D13, D6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
