File: cathode_supply.kicad_sch (KiCad schematic)
At the start: 15 parts, among them Q4 IRF540SPBF, U8 INA180A3

Commit message: A lot of work
Parts:
- removed C14 (x2), C7: 220uF 50V, Capacitor_SMD:CP_Elec_6.3x7.7, symbol MEMS_Passive:C_Elec-220uf-50V
- removed C22, C40: 10u, symbol Device:C_Small
- removed C42: 100n, symbol Device:C_Small
- removed D15: D, symbol Device:D
- removed L2: 100u, MEMS_Passive:L_Bourns_PM2110, symbol MEMS_Passive:L_100u_choke
- removed L7: L, symbol Device:L
- removed Q4: IRF540SPBF, Package_TO_SOT_SMD:TO-263-2, symbol MEMS_Discrete-semiconductor:Q_IRF540SP
- removed R29: 5m, symbol Device:R_Small
- removed U8: INA180A3, Package_TO_SOT_SMD:SOT-23-5, symbol Amplifier_Current:INA180A3
- added C14: 220uF 50V, Capacitor_SMD:CP_Elec_6.3x7.7, symbol MEMS_Passive:C_Elec-220uf-50V
- added C42, C52: 330uF 25V, Capacitor_SMD:CP_Elec_10x12.5, symbol MEMS_Passive:C_Elec-330uF-25V
- added C43, C44, C47, C54, C57: 10u, Capacitor_SMD:C_0805_2012Metric_Pad1.18x1.45mm_HandSolder, symbol Device:C_Small
- added C45, C49, C50, C53, C56: 100n, Capacitor_SMD:C_0805_2012Metric_Pad1.18x1.45mm_HandSolder, symbol Device:C_Small
- added C46: 10n, Capacitor_SMD:C_0805_2012Metric_Pad1.18x1.45mm_HandSolder, symbol Device:C_Small
- added C48, C51: ?, Capacitor_SMD:C_0805_2012Metric_Pad1.18x1.45mm_HandSolder, symbol Device:C_Small
- added C55: 100p, Capacitor_SMD:C_0805_2012Metric_Pad1.18x1.45mm_HandSolder, symbol Device:C_Small
- added L5: 220u, Inductor_SMD:L_12x12mm_H8mm, symbol MEMS_Passive:L_220u_10x10
- added L6: 8.2u, MEMS_Passive:L_Bourns_SRP7030, symbol MEMS_Passive:L_8.2u_5.9/10.2A
- added R33: 10k, Resistor_SMD:R_0805_2012Metric_Pad1.20x1.40mm_HandSolder, symbol Device:R_Small
- added R34: 1k, Resistor_SMD:R_0805_2012Metric_Pad1.20x1.40mm_HandSolder, symbol Device:R_Small
- added R35: 47k, Resistor_SMD:R_0805_2012Metric_Pad1.20x1.40mm_HandSolder, symbol Device:R_Small
- added R36, R37: ?, Resistor_SMD:R_0805_2012Metric_Pad1.20x1.40mm_HandSolder, symbol Device:R_Small
- added R38: 20m 1%, Resistor_SMD:R_2010_5025Metric_Pad1.40x2.65mm_HandSolder, symbol MEMS_Passive:R_2010_20m_1%
- added R39, R42: 8.2k, Resistor_SMD:R_0805_2012Metric_Pad1.20x1.40mm_HandSolder, symbol Device:R_Small
- added R40: 0R, Resistor_SMD:R_0805_2012Metric_Pad1.20x1.40mm_HandSolder, symbol Device:R_Small
- added R41: 100k, Resistor_SMD:R_0805_2012Metric_Pad1.20x1.40mm_HandSolder, symbol Device:R_Small
- added U10: TPS55289, MEMS_IC:TPS55289, symbol MEMS_IC:TPS55289
- R43: renamed from R30; footprint (none) -> Resistor_SMD:R_0805_2012Metric_Pad1.20x1.40mm_HandSolder
- R44: renamed from R31; footprint (none) -> Resistor_SMD:R_0805_2012Metric_Pad1.20x1.40mm_HandSolder
Connections:
- net Cathode_Supply: now also C53.2, R38.2, R41.1, U10.13 (ISN)
- net GND: now also C14.2, C42.2, C43.1, C44.1, C45.1, C46.2, C47.1, C48.2, C51.2, C52.2, C54.1, C55.1, C56.1, C57.1, R34.2, R35.2, R42.2, U10.17 (AGND), U10.2 (MODE), U10.21 (EXTVCC), U10.9 (PGND)
- net I_Monitor: now also U10.16 (CDC)
- net at F1.1: now also C14.1, L5.1
- new net: C52.1, C53.1, C54.2, C57.2, R38.1, U10.11 (VOUT), U10.12 (ISP)
- new net: C48.1, R36.1
- new net: C51.1, R37.1
- new net: C42.1, C43.2, C44.2, L5.2, R33.1, U10.7 (VIN)
- new net: R35.1, U10.6 (FSW)
- new net: C50.1, L6.2, R37.2, U10.10 (SW2)
- new net: R40.2, R41.2, R42.1
- new net: R40.1, U10.14 (FB/~{INT})
- new net: C49.1, L6.1, R36.2, U10.8 (SW1)
- new net: C49.2, U10.20 (BOOT1)
- new net: C45.2, R33.2, R34.1, U10.1 (EN/UVLO)
- new net: C55.2, R39.1, U10.15 (COMP)
- new net: C50.2, U10.19 (BOOT2)
- new net: C46.1, U10.5 (DITH/SYNC)
- new net: C56.2, R39.2
- new net +5V: C47.2, U10.18 (VCC)
- new net SCL: U10.4 (SDA)
- new net SDA: U10.3 (SCL)
Other:
- note added: "Nominal current: 1.5A -> 1.5A*20mOhm = 30mV"
- note added: "Optional snubber circuits"
- note added: "Switching frequency: 1000/(0.05*47k+35) = 420kHz Dithering frequency: 1/(2.8*47kOhm*10nF) = 760Hz"
- note added: "UVLO: 1.23V*(1+10k/1k) =13.5V"
- note removed: "Gate Drive IC"
- title: (none) -> EuroMeasure Ion Gauge Controller
- moved on the sheet: R43, R44

Commit message: Copper layout done
Parts:
- added R4, R46: 1k, Resistor_SMD:R_0805_2012Metric_Pad1.20x1.40mm_HandSolder, symbol Device:R_Small
Connections:
- net SCL: now also R46.2
- net SDA: now also R4.2
- net 15V_Filtered: now reaches C14.1, F1.1, L5.1
- net SW1: now reaches C49.1, L6.1, R36.2, U10.8 (SW1)
- new net +3.3V: R4.1, R46.1
Changed lines of the file:
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@@
     (rev "1.0.0")
   )
+  (junction (at 80.01 116.84) (diameter 0) (color 0 0 0 0)
+  )
   (junction (at 113.03 105.41) (diameter 0) (color 0 0 0 0)
   )
+  (junction (at 80.01 107.95) (diameter 0) (color 0 0 0 0)
+  )
   (junction (at 180.34 97.79) (diameter 0) (color 0 0 0 0)
   )
@@
   (junction (at 208.28 97.79) (diameter 0) (color 0 0 0 0)
   )
+  (junction (at 83.82 119.38) (diameter 0) (color 0 0 0 0)
+  )
   (junction (at 177.8 69.85) (diameter 0) (color 0 0 0 0)
   )
@@
     (stroke (width 0) (type default))
   )
-  (wire (pts (xy 124.46 115.57) (xy 128.27 115.57))
+  (wire (pts (xy 76.2 119.38) (xy 83.82 119.38))
     (stroke (width 0) (type default))
   )
@@
     (stroke (width 0) (type default))
   )
-  (wire (pts (xy 124.46 113.03) (xy 128.27 113.03))
+  (wire (pts (xy 83.82 107.95) (xy 83.82 109.22))
+    (stroke (width 0) (type default))
+  )
+  (wire (pts (xy 76.2 116.84) (xy 80.01 116.84))
     (stroke (width 0) (type default))
   )
@@
     (stroke (width 0) (type default))
   )
+  (wire (pts (xy 123.19 116.84) (xy 123.19 113.03))
+    (stroke (width 0) (type default))
+  )
   (wire (pts (xy 85.09 92.71) (xy 85.09 88.9))
     (stroke (width 0) (type default))
   )
+  (wire (pts (xy 80.01 107.95) (xy 83.82 107.95))
+    (stroke (width 0) (type default))
+  )
   (wire (pts (xy 182.88 130.81) (xy 182.88 132.08))
     (stroke (width 0) (type default))
@@
     (stroke (width 0) (type default))
   )
+  (wire (pts (xy 80.01 116.84) (xy 123.19 116.84))
+    (stroke (width 0) (type default))
+  )
   (wire (pts (xy 107.95 80.01) (xy 127 80.01))
     (stroke (width 0) (type default))
@@
     (stroke (width 0) (type default))
   )
+  (wire (pts (xy 80.01 114.3) (xy 80.01 116.84))
+    (stroke (width 0) (type default))
+  )
+  (wire (pts (xy 125.73 119.38) (xy 125.73 115.57))
+    (stroke (width 0) (type default))
+  )
   (wire (pts (xy 107.95 111.76) (xy 107.95 113.03))
     (stroke (width 0) (type default))
@@
     (stroke (width 0) (type default))
   )
+  (wire (pts (xy 83.82 114.3) (xy 83.82 119.38))
+    (stroke (width 0) (type default))
+  )
   (wire (pts (xy 135.89 83.82) (xy 135.89 85.09))
     (stroke (width 0) (type default))
@@
     (stroke (width 0) (type default))
   )
+  (wire (pts (xy 80.01 106.68) (xy 80.01 107.95))
+    (stroke (width 0) (type default))
+  )
   (wire (pts (xy 208.28 99.06) (xy 208.28 97.79))
     (stroke (width 0) (type default))
@@
     (stroke (width 0) (type default))
   )
+  (wire (pts (xy 123.19 113.03) (xy 128.27 113.03))
+    (stroke (width 0) (type default))
+  )
   (wire (pts (xy 185.42 80.01) (xy 185.42 78.74))
     (stroke (width 0) (type default))
@@
     (stroke (width 0) (type default))
   )
+  (wire (pts (xy 80.01 107.95) (xy 80.01 109.22))
+    (stroke (width 0) (type default))
+  )
   (wire (pts (xy 107.95 105.41) (xy 113.03 105.41))
     (stroke (width 0) (type default))
@@
     (stroke (width 0) (type default))
   )
+  (wire (pts (xy 125.73 115.57) (xy 128.27 115.57))
+    (stroke (width 0) (type default))
+  )
   (wire (pts (xy 135.89 77.47) (xy 135.89 78.74))
     (stroke (width 0) (type default))
@@
   )
   (wire (pts (xy 177.8 124.46) (xy 177.8 132.08))
+    (stroke (width 0) (type default))
+  )
+  (wire (pts (xy 83.82 119.38) (xy 125.73 119.38))
     (stroke (width 0) (type default))
   )
@@
     (effects (font (size 1.27 1.27)) (justify left bottom))
   )
+  (label "15V_Filtered" (at 72.39 80.01 90) (fields_autoplaced)
+    (effects (font (size 1.27 1.27)) (justify left bottom))
+  )
+  (label "SW1" (at 140.97 83.82 90) (fields_autoplaced)
+    (effects (font (size 1.27 1.27)) (justify left bottom))
+  )
   (hierarchical_label "I_Monitor" (shape output) (at 166.37 123.19 0) (fields_autoplaced)
     (effects (font (size 1.27 1.27)) (justify left))
@@
     (effects (font (size 1.27 1.27)) (justify left))
   )
-  (hierarchical_label "SCL" (shape input) (at 124.46 115.57 180) (fields_autoplaced)
+  (hierarchical_label "SCL" (shape input) (at 76.2 119.38 180) (fields_autoplaced)
     (effects (font (size 1.27 1.27)) (justify right))
   )
-  (hierarchical_label "SDA" (shape bidirectional) (at 124.46 113.03 180) (fields_autoplaced)
+  (hierarchical_label "SDA" (shape bidirectional) (at 76.2 116.84 180) (fields_autoplaced)
     (effects (font (size 1.27 1.27)) (justify right))
   )
@@
       (effects (font (size 1.27 1.27)) hide)
     )
-    (property "Value" "GND" (at 113.03 116.84 0)
+    (property "Value" "GND" (at 116.84 114.3 0)
       (effects (font (size 1.27 1.27)))
     )
@@
     )
   )
+  (symbol (lib_id "Device:R_Small") (at 83.82 111.76 0) (mirror y) (unit 1)
+    (in_bom yes) (on_board yes) (dnp no) (fields_autoplaced)
+    (property "Reference" "R46" (at 86.36 110.49 0)
+      (effects (font (size 1.27 1.27)) (justify right))
+    )
+    (property "Value" "1k" (at 86.36 113.03 0)
+      (effects (font (size 1.27 1.27)) (justify right))
+    )
+    (property "Footprint" "Resistor_SMD:R_0805_2012Metric_Pad1.20x1.40mm_HandSolder" (at 83.82 111.76 0)
+      (effects (font (size 1.27 1.27)) hide)
+    )
+    (property "Datasheet" "~" (at 83.82 111.76 0)
+      (effects (font (size 1.27 1.27)) hide)
+    )
+    (pin "1")
+    (pin "2")
+    (instances
+      (project "EuroMeasure-IonGaugeController"
+        (path "/9c84a828-ebcc-4f88-b5cc-11be4f5044ad/192a135a-32d5-437a-a3cf-556f2261accf"
+          (reference "R46") (unit 1)
+        )
+      )
+    )
+  )
   (symbol (lib_id "Device:R_Small") (at 187.96 118.11 90) (unit 1)
     (in_bom yes) (on_board yes) (dnp no) (fields_autoplaced)
@@
       (effects (font (size 1.27 1.27)) hide)
     )
-    (property "Value" "GND" (at 107.95 116.84 0)
+    (property "Value" "GND" (at 104.14 114.3 0)
       (effects (font (size 1.27 1.27)))
     )
@@
     )
   )
+  (symbol (lib_id "power:+3.3V") (at 80.01 106.68 0) (unit 1)
+    (in_bom yes) (on_board yes) (dnp no) (fields_autoplaced)
+    (property "Reference" "#PWR055" (at 80.01 110.49 0)
+      (effects (font (size 1.27 1.27)) hide)
+    )
+    (property "Value" "+3.3V" (at 80.01 101.6 0)
+      (effects (font (size 1.27 1.27)))
+    )
+    (property "Footprint" "" (at 80.01 106.68 0)
+      (effects (font (size 1.27 1.27)) hide)
+    )
+    (property "Datasheet" "" (at 80.01 106.68 0)
+      (effects (font (size 1.27 1.27)) hide)
+    )
+    (pin "1")
+    (instances
+      (project "EuroMeasure-IonGaugeController"
+        (path "/9c84a828-ebcc-4f88-b5cc-11be4f5044ad/abf38db6-df21-42a4-a2d8-4fd7d247b99e"
+          (reference "#PWR055") (unit 1)
+        )
+        (path "/9c84a828-ebcc-4f88-b5cc-11be4f5044ad"
+          (reference "#PWR011") (unit 1)
+        )
+        (path "/9c84a828-ebcc-4f88-b5cc-11be4f5044ad/192a135a-32d5-437a-a3cf-556f2261accf"
+          (reference "#PWR0113") (unit 1)
+        )
+      )
+      (project "EuroMeasure-Generator"
+        (path "/c0f57af1-51e3-4b1b-8afb-67a4c2f2a5dd/5c32201f-9cee-4b13-85be-b08d669b436d"
+          (reference "#PWR0925") (unit 1)
+        )
+      )
+    )
+  )
   (symbol (lib_id "Device:C_Small") (at 177.8 76.2 0) (mirror x) (unit 1)
     (in_bom yes) (on_board yes) (dnp no)
@@
         )
       )
+    )
+  )
+  (symbol (lib_id "Device:R_Small") (at 80.01 111.76 0) (mirror y) (unit 1)
+    (in_bom yes) (on_board yes) (dnp no)
+    (property "Reference" "R4" (at 77.47 110.49 0)
+      (effects (font (size 1.27 1.27)) (justify left))
+    )
+    (property "Value" "1k" (at 77.47 113.03 0)
+      (effects (font (size 1.27 1.27)) (justify left))
+    )
+    (property "Footprint" "Resistor_SMD:R_0805_2012Metric_Pad1.20x1.40mm_HandSolder" (at 80.01 111.76 0)
+      (effects (font (size 1.27 1.27)) hide)
+    )
+    (property "Datasheet" "~" (at 80.01 111.76 0)
+      (effects (font (size 1.27 1.27)) hide)
+    )
+    (pin "1")
+    (pin "2")
+    (instances
+      (project "EuroMeasure-IonGaugeController"
+        (path "/9c84a828-ebcc-4f88-b5cc-11be4f5044ad/192a135a-32d5-437a-a3cf-556f2261accf"
+          (reference "R4") (unit 1)
+        )
+      )

Commit message: Revision 1.1.0. DRC clean
Parts:
- added R47: 0R, Resistor_SMD:R_0805_2012Metric_Pad1.20x1.40mm_HandSolder, symbol Device:R_Small
- R40: now not fitted
Connections:
- net GND: now also R47.2
- net 15V_FILTERED: now reaches C42.1, C43.2, C44.2, L5.2, R33.1, U10.7 (VIN)
- net at C46.1, U10.5 (DITH/SYNC): now also R47.1
- net +15V renamed 15V_IN
- net 15V_Filtered: no longer names the net of C14.1, F1.1, L5.1
- net Cathode_Supply renamed +
- net I_Monitor renamed I
- net U_Monitor renamed V
Other:
- note added: "Gain: 1k/(1k+10k) =0.091"
- note added: "Place either of the two components"
- note added: "Undervoltage lockout: 1.23V*(1+10k/1k) =13.5V"
- note added: "Vout = Vref*(1+100k/8.2k)"
- note removed: "UVLO: 1.23V*(1+10k/1k) =13.5V"
- moved on the sheet: C14, C42, C43, C44, F1, L5

Commit message: Everything clear. Gerbers generated
Parts:
- C33: renamed from C48; value ? -> ~
- C36: renamed from C51; value ? -> ~
- R30: renamed from R36; value ? -> ~
- R31: renamed from R37; value ? -> ~
- renumbered C42 to C27, C43 to C28, C44 to C29, C45 to C30, C46 to C31, C47 to C32, C49 to C34, C50 to C35, C52 to C37, C53 to C38, C54 to C39, C55 to C40, C56 to C41, C57 to C42, L5 to L4, L6 to L5, R4 to R24, R46 to R25, R47 to R26, R33 to R27, R34 to R28, R35 to R29, R38 to R32, R39 to R33, R40 to R34, R41 to R35, R42 to R36, R43 to R37, R44 to R38, U10 to U7
