File: grid_current_measurement.kicad_sch (KiCad schematic)
At the start: 5 parts

Commit message: Everything clear. Gerbers generated
Parts:
- renumbered C17 to C52, DZ2 to DZ3, R11 to R45, R12 to R46, R13 to R47
Changed lines of the file:
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@@
   (symbol (lib_id "power:GND") (at 134.62 102.87 0) (mirror y) (unit 1)
     (in_bom yes) (on_board yes) (dnp no) (fields_autoplaced)
-    (property "Reference" "#PWR034" (at 134.62 109.22 0)
+    (property "Reference" "#PWR087" (at 134.62 109.22 0)
       (effects (font (size 1.27 1.27)) hide)
     )
@@
       (project "EuroMeasure-IonGaugeController"
         (path "/9c84a828-ebcc-4f88-b5cc-11be4f5044ad/44c02725-ef07-40c2-83a3-a15b117f305b"
-          (reference "#PWR034") (unit 1)
+          (reference "#PWR087") (unit 1)
         )
       )
@@
   (symbol (lib_id "MEMS_Passive:R_0805_100R_0.1%_5PPM") (at 134.62 90.17 0) (unit 1)
     (in_bom yes) (on_board yes) (dnp no) (fields_autoplaced)
-    (property "Reference" "R11" (at 132.08 88.9 0)
+    (property "Reference" "R45" (at 132.08 88.9 0)
       (effects (font (size 1.27 1.27)) (justify right))
     )
@@
       (project "EuroMeasure-IonGaugeController"
         (path "/9c84a828-ebcc-4f88-b5cc-11be4f5044ad/44c02725-ef07-40c2-83a3-a15b117f305b"
-          (reference "R11") (unit 1)
+          (reference "R45") (unit 1)
         )
       )
@@
   (symbol (lib_id "MEMS_Passive:R_0805_100R_0.1%_5PPM") (at 134.62 96.52 0) (unit 1)
     (in_bom yes) (on_board yes) (dnp no) (fields_autoplaced)
-    (property "Reference" "R12" (at 132.08 95.25 0)
+    (property "Reference" "R46" (at 132.08 95.25 0)
       (effects (font (size 1.27 1.27)) (justify right))
     )
@@
       (project "EuroMeasure-IonGaugeController"
         (path "/9c84a828-ebcc-4f88-b5cc-11be4f5044ad/44c02725-ef07-40c2-83a3-a15b117f305b"
-          (reference "R12") (unit 1)
+          (reference "R46") (unit 1)
         )
       )
@@
   (symbol (lib_id "power:GND") (at 148.59 102.87 0) (mirror y) (unit 1)
     (in_bom yes) (on_board yes) (dnp no) (fields_autoplaced)
-    (property "Reference" "#PWR035" (at 148.59 109.22 0)
+    (property "Reference" "#PWR088" (at 148.59 109.22 0)
       (effects (font (size 1.27 1.27)) hide)
     )
@@
       (project "EuroMeasure-IonGaugeController"
         (path "/9c84a828-ebcc-4f88-b5cc-11be4f5044ad/44c02725-ef07-40c2-83a3-a15b117f305b"
-          (reference "#PWR035") (unit 1)
+          (reference "#PWR088") (unit 1)
         )
       )
@@
   (symbol (lib_id "MEMS_Discrete-semiconductor:D_Zener_2V4_dual_MMBZ5221BS") (at 158.75 97.79 270) (unit 2)
     (in_bom yes) (on_board yes) (dnp no) (fields_autoplaced)
-    (property "Reference" "DZ2" (at 161.29 96.52 90)
+    (property "Reference" "DZ3" (at 161.29 96.52 90)
       (effects (font (size 1.27 1.27)) (justify left))
     )
@@
       (project "EuroMeasure-IonGaugeController"
         (path "/9c84a828-ebcc-4f88-b5cc-11be4f5044ad/44c02725-ef07-40c2-83a3-a15b117f305b"
-          (reference "DZ2") (unit 2)
+          (reference "DZ3") (unit 2)
         )
       )
@@
   (symbol (lib_id "power:GND") (at 158.75 102.87 0) (mirror y) (unit 1)
     (in_bom yes) (on_board yes) (dnp no) (fields_autoplaced)
-    (property "Reference" "#PWR036" (at 158.75 109.22 0)
+    (property "Reference" "#PWR089" (at 158.75 109.22 0)
       (effects (font (size 1.27 1.27)) hide)
     )
@@
       (project "EuroMeasure-IonGaugeController"
         (path "/9c84a828-ebcc-4f88-b5cc-11be4f5044ad/44c02725-ef07-40c2-83a3-a15b117f305b"
-          (reference "#PWR036") (unit 1)
+          (reference "#PWR089") (unit 1)
         )
       )
@@
   (symbol (lib_id "Device:R_Small") (at 142.24 83.82 90) (unit 1)
     (in_bom yes) (on_board yes) (dnp no) (fields_autoplaced)
-    (property "Reference" "R13" (at 142.24 77.47 90)
+    (property "Reference" "R47" (at 142.24 77.47 90)
       (effects (font (size 1.27 1.27)))
     )
@@
       (project "EuroMeasure-IonGaugeController"
         (path "/9c84a828-ebcc-4f88-b5cc-11be4f5044ad/44c02725-ef07-40c2-83a3-a15b117f305b"
-          (reference "R13") (unit 1)
+          (reference "R47") (unit 1)
         )
       )
@@
   (symbol (lib_id "Device:C_Small") (at 148.59 92.71 0) (unit 1)
     (in_bom yes) (on_board yes) (dnp no)
-    (property "Reference" "C17" (at 152.4 92.71 90)
+    (property "Reference" "C52" (at 152.4 92.71 90)
       (effects (font (size 1.27 1.27)))
     )
@@
       (project "EuroMeasure-IonGaugeController"
         (path "/9c84a828-ebcc-4f88-b5cc-11be4f5044ad/44c02725-ef07-40c2-83a3-a15b117f305b"
-          (reference "C17") (unit 1)
+          (reference "C52") (unit 1)
         )
       )
@@
   (symbol (lib_id "MEMS_Discrete-semiconductor:D_Zener_2V4_dual_MMBZ5221BS") (at 158.75 88.9 90) (unit 1)
     (in_bom yes) (on_board yes) (dnp no) (fields_autoplaced)
-    (property "Reference" "DZ2" (at 161.29 87.63 90)
+    (property "Reference" "DZ3" (at 161.29 87.63 90)
       (effects (font (size 1.27 1.27)) (justify right))
     )
@@
       (project "EuroMeasure-IonGaugeController"
         (path "/9c84a828-ebcc-4f88-b5cc-11be4f5044ad/44c02725-ef07-40c2-83a3-a15b117f305b"
-          (reference "DZ2") (unit 1)
-        )
-      )
+          (reference "DZ3") (unit 1)
+        )
+      )
