File: grid_supply.kicad_sch (KiCad schematic)
At the start: 41 parts, among them K1 UD2-5NU, Q4 IRF540SPBF, Q5 FZT1053A, Q6 FZT1053A, U1 TL072

Commit message: A lot of work
Parts:
- removed C11: 100n, Capacitor_SMD:C_0805_2012Metric_Pad1.18x1.45mm_HandSolder, symbol Device:C_Small
- removed C14, C7: 220uF 50V, Capacitor_SMD:CP_Elec_6.3x7.7, symbol MEMS_Passive:C_Elec-220uf-50V
- removed D12: 6V3, Diode_SMD:D_MELF, symbol MEMS_Discrete-semiconductor:D_Zener_6V3_TZMB3V6-GS08
- removed D6: D_Zener_3.2V, symbol Device:D_Zener
- removed F1: Polyfuse 2A, MEMS_Passive:Fuse_Littlefuse_3425L, symbol MEMS_Protection:Polyfuse-2A-60V-3425L200/60MR
- removed L2: 100u, MEMS_Passive:L_Bourns_PM2110, symbol MEMS_Passive:L_100u_choke
- removed R11: 10k, symbol Device:R_Small
- removed R16: 820 0.5W, Resistor_SMD:R_1210_3225Metric_Pad1.30x2.65mm_HandSolder, symbol MEMS_Passive:R_820Ohm_1210
- added C28, C30: 10u, Capacitor_SMD:C_0805_2012Metric_Pad1.18x1.45mm_HandSolder, symbol Device:C_Small
- added unit 2 of DZ2
- added R11, R12: 100R 0.1% 5PPM, Resistor_SMD:R_0805_2012Metric_Pad1.20x1.40mm_HandSolder, symbol MEMS_Passive:R_0805_100R_0.1%_5PPM
- added R45: R_1210_820Ohm, Resistor_SMD:R_1210_3225Metric_Pad1.30x2.65mm_HandSolder, symbol MEMS_Passive:R_1210_820Ohm
- added U3: 3.0V, Package_TO_SOT_SMD:SOT-23, symbol MEMS_IC:LM4040-3.0
- C9: value 100n -> 10n; footprint Capacitor_SMD:C_0805_2012Metric -> Capacitor_SMD:C_0805_2012Metric_Pad1.18x1.45mm_HandSolder; now fitted
- R11: value ? -> 10k
- R9: value 33k -> 30k
Connections:
- net +15V: now also C11.2
- net +5V: now also R45.2; no longer K1.4
- net -15V: now also C11.1
- net GND: now also C11.1, C11.2, C28.1, C30.1, DZ2.3 (K), R12.2, U3.2 (A)
- net GNDD: now also R16.1, R11.1; no longer U1.6 (-)
- net I_Monitor: now also DZ2.6 (K)
- net heatsink_1: now also C18.1
- net heatsink_2: now also C18.2
- net at C11.2, R11.2, U1.5 (+): now also U3.1 (K)
- net at FL2.2, Q6.1 (B): now also R45.1
- net at FL2.3: now also K1.5, C28.2, C30.2
- net at U1.7: now also U1.6 (-); no longer R16.1
- new net: R11.2, R12.1
- new net: DZ2.1 (A), DZ2.4 (A)
- new net +5VL: K1.4
Other:
- note added: "(5V-3V)/10k = 200uA"
- note added: "0.2V/mA"
- note added: "3V*(1+2M/30k) =~ 200V"
- moved on the sheet: D5, R13, R16, R9

Commit message: Copper layout done
Connections:
- net 5V_Lockouted: now reaches C28.2, C30.2, FL2.3, K1.5
Changed lines of the file:
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@@
     (effects (font (size 1.27 1.27)) (justify right bottom))
+  )
+  (label "5V_Lockouted" (at 74.93 67.31 0) (fields_autoplaced)
+    (effects (font (size 1.27 1.27)) (justify left bottom))
   )
   (global_label "~{LOCKOUT}" (shape input) (at 52.07 67.31 90) (fields_autoplaced)

Commit message: Final 1.0.0 version
Parts:
- U1: MPN (none) -> TL082IDRQ1
Changed lines of the file:
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@@
     )
   )
-  (symbol (lib_name "TL082IDRQ1_1") (lib_id "MEMS_IC:TL082IDRQ1") (at 146.05 168.91 180) (unit 2)
+  (symbol (lib_id "MEMS_IC:TL082IDRQ1") (at 146.05 168.91 180) (unit 2)
     (in_bom yes) (on_board yes) (dnp no)
     (property "Reference" "U1" (at 142.24 172.72 0)
@@
     )
     (property "Mouser" "595-TL082IDRQ1" (at 146.05 168.91 0)
+      (effects (font (size 1.27 1.27)) hide)
+    )
+    (property "MPN" "TL082IDRQ1" (at 146.05 168.91 0)
       (effects (font (size 1.27 1.27)) hide)
     )
@@
     )
   )
-  (symbol (lib_name "TL082IDRQ1_1") (lib_id "MEMS_IC:TL082IDRQ1") (at 158.75 109.22 180) (unit 2)
+  (symbol (lib_id "MEMS_IC:TL082IDRQ1") (at 158.75 109.22 180) (unit 2)
     (in_bom yes) (on_board yes) (dnp no)
     (property "Reference" "U1" (at 154.94 113.03 0)
@@
     )
     (property "Mouser" "595-TL082IDRQ1" (at 158.75 109.22 0)
+      (effects (font (size 1.27 1.27)) hide)
+    )
+    (property "MPN" "TL082IDRQ1" (at 158.75 109.22 0)
       (effects (font (size 1.27 1.27)) hide)
     )
@@
     )
   )
-  (symbol (lib_name "TL082IDRQ1_1") (lib_id "MEMS_IC:TL082IDRQ1") (at 113.03 168.91 180) (unit 2)
+  (symbol (lib_id "MEMS_IC:TL082IDRQ1") (at 113.03 168.91 180) (unit 2)
     (in_bom yes) (on_board yes) (dnp no)
     (property "Reference" "U1" (at 109.22 172.72 0)
@@
       (effects (font (size 1.27 1.27)) hide)
     )
+    (property "MPN" "TL082IDRQ1" (at 113.03 168.91 0)
+      (effects (font (size 1.27 1.27)) hide)
+    )

Commit message: Revision 1.1.0. DRC clean
Parts:
- removed C17: 1n 1210, Capacitor_SMD:C_1210_3225Metric_Pad1.33x2.70mm_HandSolder, symbol MEMS_Passive:C_1210_1n
- removed C9: 10n, Capacitor_SMD:C_0805_2012Metric_Pad1.18x1.45mm_HandSolder, symbol Device:C_Small
- removed unit 2 of DZ2
- removed R11, R12: 100R 0.1% 5PPM, Resistor_SMD:R_0805_2012Metric_Pad1.20x1.40mm_HandSolder, symbol MEMS_Passive:R_0805_100R_0.1%_5PPM
- removed R15: 1k 0.5W, Resistor_SMD:R_1210_3225Metric_Pad1.30x2.65mm_HandSolder, symbol MEMS_Passive:R_1210_1k
- removed R16: 1k, Resistor_SMD:R_0805_2012Metric, symbol Device:R_Small
- added C13: 1n X7R, Capacitor_SMD:C_1210_3225Metric_Pad1.33x2.70mm_HandSolder, symbol MEMS_Passive:C_1210_1nF_1000V_X7R
- added R7: 1k 0.5W, Resistor_SMD:R_1210_3225Metric_Pad1.30x2.65mm_HandSolder, symbol MEMS_Passive:R_1210_1k_5%
- renumbered C28 to C7, C30 to C8
Connections:
- net GND: no longer C11.1, U3.2 (A)
- net GNDD: now also C11.1, U3.2 (A)
- net heatsink_3: now also L3.1, Q5.3 (E), Q6.3 (E); no longer L3.2, Q4.2 (D)
- net GRID_AC0: now reaches D6.2 (A), D7.1 (K), FL2.9
- net GRID_Unfiltered: now reaches C16.1, D6.1 (K), D9.1 (K)
- net GRID_Unfiltered: now also C13.1, R7.1
- net GRID_AC1: now reaches D8.1 (K), D9.2 (A), FL2.8
- net at R14.1: now also C13.2
- net +5VL renamed 5V_IN
- net 200V_Grid_Supply renamed +
- net +: now also R7.2
- new net heatsink_4: L3.2, Q4.2 (D)
Other:
- note added: "AC Feedback"
- note added: "Bias current:"
- note added: "DANGER! HAZARDOUS VOLTAGE"
- note added: "DC Feedback"
- note added: "To change output voltage adjust the R9-R10 divider, for example:"
- note added: "Unused OP-amp"
- note removed: "0.2V/mA"
- moved on the sheet: C11, C15, C16, C18, C7, C8, C9, D6, D7, D8, D9, DZ2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

Commit message: Everything clear. Gerbers generated
Parts:
- FL2: value ~ -> FL2015-4L
- renumbered C13 to C12, R7 to R11, R45 to R8
