File: psu.kicad_sch (KiCad schematic)
At the start: 11 parts, among them U4 AZ1117-3V3

Commit message: Everything clear. Gerbers generated
Parts:
- TP17: symbol Connector:TestPoint -> MEMS_Other:TP_1mm_via; now left out of the parts list
- renumbered C18 to C53, C19 to C54, C1 to C55, C2 to C56, C20 to C57, C21 to C58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
