File: EuroMeasure-IonGaugeController.kicad_sch (KiCad schematic)
At the start: 5 parts

Commit message: Rename to Ion Gauge Controller
Other:
- title: EuroMeasure blank module -> EuroMeasure Ion Gauge Controller
Changed lines of the file:
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@@
   (paper "A4")
   (title_block
-    (title "EuroMeasure blank module")
+    (title "EuroMeasure Ion Gauge Controller")
+    (date "2023-10-17")
+    (rev "1.0.0")
   )
   (bus_alias "ADC_ISO" (members "RESET" "DRDY" "CS" "SCLK" "DIN" "DOUT" "CLK"))
@@
     (pin "1")
     (instances
-      (project "EuroMeasure-Module"
+      (project "EuroMeasure-IonGaugeController"
         (path "/9c84a828-ebcc-4f88-b5cc-11be4f5044ad/abf38db6-df21-42a4-a2d8-4fd7d247b99e"
           (reference "TP909") (unit 1)
@@
     (pin "1")
     (instances
-      (project "EuroMeasure-Module"
+      (project "EuroMeasure-IonGaugeController"
         (path "/9c84a828-ebcc-4f88-b5cc-11be4f5044ad/abf38db6-df21-42a4-a2d8-4fd7d247b99e"
           (reference "TP908") (unit 1)
@@
     (pin "1")
     (instances
-      (project "EuroMeasure-Module"
+      (project "EuroMeasure-IonGaugeController"
         (path "/9c84a828-ebcc-4f88-b5cc-11be4f5044ad/abf38db6-df21-42a4-a2d8-4fd7d247b99e"
           (reference "TP910") (unit 1)
@@
     (pin "1")
     (instances
-      (project "EuroMeasure-Module"
+      (project "EuroMeasure-IonGaugeController"
         (path "/9c84a828-ebcc-4f88-b5cc-11be4f5044ad/abf38db6-df21-42a4-a2d8-4fd7d247b99e"
           (reference "TP906") (unit 1)
@@
     (pin "1")
     (instances
-      (project "EuroMeasure-Module"
+      (project "EuroMeasure-IonGaugeController"
         (path "/9c84a828-ebcc-4f88-b5cc-11be4f5044ad/abf38db6-df21-42a4-a2d8-4fd7d247b99e"
           (reference "TP907") (unit 1)
@@
     )
     (instances
-      (project "EuroMeasure-Module"
+      (project "EuroMeasure-IonGaugeController"
         (path "/9c84a828-ebcc-4f88-b5cc-11be4f5044ad" (page "3"))
       )

Commit message: First schematic draft
Parts:
- added C1, C2, C3: 10u, Capacitor_SMD:C_0805_2012Metric_Pad1.18x1.45mm_HandSolder, symbol Device:C_Small
- added C4: 100n, Capacitor_SMD:C_0805_2012Metric_Pad1.18x1.45mm_HandSolder, symbol Device:C_Small
- added J1: Conn_01x04, symbol Connector_Generic:Conn_01x04
- added R1: 1, Resistor_SMD:R_0805_2012Metric_Pad1.20x1.40mm_HandSolder, symbol Device:R_Small
- added R2: 10, Resistor_SMD:R_0805_2012Metric_Pad1.20x1.40mm_HandSolder, symbol Device:R_Small
- added TP906: ADC_DRDY, MEMS_Custom:TestPoint_Pad_D1.0mm, symbol Connector:TestPoint
- added TP907: ADC_RESET, MEMS_Custom:TestPoint_Pad_D1.0mm, symbol Connector:TestPoint
- added TP908: ADC_CS, MEMS_Custom:TestPoint_Pad_D1.0mm, symbol Connector:TestPoint
- added U1: ADS131M04-WQFN, Package_DFN_QFN:WQFN-20-1EP_3x3mm_P0.4mm_EP1.7x1.7mm, symbol MEMS_IC:ADS131M04-WQFN
- added X1: 8.192MHz, Oscillator:Oscillator_SMD_ECS_2520MV-xxx-xx-4Pin_2.5x2.0mm, symbol MEMS_IC:ECS-2520MVLC-081.92-CN-TR_oscillator_8.192MHZ
Connections:
- net EuroMeasure/SPI1_MISO renamed DOUT
- net DOUT: now also U1.13 (DOUT)
- net EuroMeasure/SPI1_MOSI renamed DIN
- net DIN: now also U1.14 (DIN)
- net EuroMeasure/SPI1_SCK renamed SCLK
- net SCLK: now also U1.12 (SCLK)
- new net: C3.1, R2.1, U1.18 (DVDD)
- new net: C1.2, R1.1, U1.19 (AVDD)
- new net: C2.1, U1.16 (CAP)
- new net +3V3: C4.2, R1.2, R2.2, X1.4 (VDD)
- new net AIN0N: U1.2 (AIN0N)
- new net AIN1N: U1.3 (AIN1N)
- new net AIN2N: U1.6 (AIN2N)
- new net AIN3N: U1.7 (AIN3N)
- new net Anode: J1.2 (Pin_2)
- new net CLK: U1.15 (CLKIN), X1.3 (OUT)
- new net CS: TP908.1, U1.10 (~{CS})
- new net Cathode: J1.3 (Pin_3)
- new net DRDY: TP906.1, U1.11 (~{DRDY})
- new net GND: C1.1, C2.2, C3.2, J1.4 (Pin_4), U1.1 (AIN0P), U1.17 (DGND), U1.20 (AGND), U1.21 (THERMAL(AGND)), U1.4 (AIN1P), U1.5 (AIN2P), U1.8 (AIN3P)
- new net GNDF: C4.1, X1.2 (GND)
- new net Grid: J1.1 (Pin_1)
- new net RESET: TP907.1, U1.9 (~{SYNC}/~{RESET})
- no-connect marks 29 -> 26
Other:
- added sheet Anode Supply (anode_supply.kicad_sch)
- added sheet Cathode Supply (cathode_supply.kicad_sch)
- added sheet Grid Supply (grid_supply.kicad_sch)
- note added: "Overkill but already used elsewhere and supported by software"
- moved on the sheet: TP906, TP907, TP908, TP909, TP910

Commit message: A lot of work
Parts:
- added C1, C2: 220uF 50V, Capacitor_SMD:CP_Elec_6.3x7.7, symbol MEMS_Passive:C_Elec-220uf-50V
- added F1: Polyfuse 2A, MEMS_Passive:Fuse_Littlefuse_3425L, symbol MEMS_Protection:Polyfuse-2A-60V-3425L200/60MR
- added L1: 220u, Inductor_SMD:L_12x12mm_H8mm, symbol MEMS_Passive:L_220u_10x10
- added TP906: Anode_I, MEMS_Custom:TestPoint_Pad_D1.0mm, symbol Connector:TestPoint
- added TP906: Grid_I, MEMS_Custom:TestPoint_Pad_D1.0mm, symbol Connector:TestPoint
- added TP906: Cathode_I, MEMS_Custom:TestPoint_Pad_D1.0mm, symbol Connector:TestPoint
- added TP906: Cathode_V, MEMS_Custom:TestPoint_Pad_D1.0mm, symbol Connector:TestPoint
- J1: footprint (none) -> Connector_Dsub:DSUB-9_Female_Horizontal_P2.77x2.54mm_EdgePinOffset9.40mm
- renumbered C1 to C3, C2 to C4, C3 to C5, C4 to C6
Connections:
- net GNDF is gone; now on net GND: C6.1, X1.2 (GND)
- net AIN0N: now also TP906.1
- net AIN1N: now also TP906.1
- net AIN2N: now also TP906.1
- net AIN3N: now also TP906.1
- net GND: now also C1.2, C2.2
- net +3V3 renamed +3.3V
- net EuroMeasure/SCL_INT renamed Cathode Supply/SCL
- net EuroMeasure/SDA_INT renamed Cathode Supply/SDA
- new net: C1.1, F1.1, L1.1
- new net +5V: F1.2
- new net +5VL: C2.1, L1.2
- no-connect marks 26 -> 27
Other:
- sheet Anode Supply ports: added -25V_Anode_Supply; removed -25V_Grid_Supply
- sheet Cathode Supply ports: added SCL, SDA; removed Control
- note added: "-1.2V - 1.2V range"
- moved on the sheet: C6

Commit message: Copper layout done
Parts:
- removed J1: Conn_01x04, Connector_Dsub:DSUB-9_Female_Horizontal_P2.77x2.54mm_EdgePinOffset9.40mm, symbol Connector_Generic:Conn_01x04
- added J1: Conn_02x05_Odd_Even, Connector_IDC:IDC-Header_2x05_P2.54mm_Vertical, symbol Connector_Generic:Conn_02x05_Odd_Even
Connections:
- net Anode: now also J1.2 (Pin_2)
- net Cathode: now also J1.7 (Pin_7), J1.8 (Pin_8)
- net GND: now also J1.10 (Pin_10), J1.9 (Pin_9)
- net Grid: now also J1.3 (Pin_3)
- no-connect marks 27 -> 31
Other:
- moved on the sheet: TP906

Commit message: Final 1.0.0 version
Parts:
- J1: MPN (none) -> NO_MPN
Changed lines of the file:
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@@
+      (effects (font (size 1.27 1.27)) hide)
+    )
+    (property "MPN" "NO_MPN" (at 125.73 138.43 0)
       (effects (font (size 1.27 1.27)) hide)
     )

Commit message: Revision 1.1.0. DRC clean
Parts:
- removed C1, C2: 220uF 50V, Capacitor_SMD:CP_Elec_6.3x7.7, symbol MEMS_Passive:C_Elec-220uf-50V
- removed C3, C4, C5: 10u, Capacitor_SMD:C_0805_2012Metric_Pad1.18x1.45mm_HandSolder, symbol Device:C_Small
- removed C6: 100n, Capacitor_SMD:C_0805_2012Metric_Pad1.18x1.45mm_HandSolder, symbol Device:C_Small
- removed F1: Polyfuse 2A, MEMS_Passive:Fuse_Littlefuse_3425L, symbol MEMS_Protection:Polyfuse-2A-60V-3425L200/60MR
- removed J1: Conn_02x05_Odd_Even, Connector_IDC:IDC-Header_2x05_P2.54mm_Vertical, symbol Connector_Generic:Conn_02x05_Odd_Even
- removed L1: 220u, Inductor_SMD:L_12x12mm_H8mm, symbol MEMS_Passive:L_220u_10x10
- removed R1: 1, Resistor_SMD:R_0805_2012Metric_Pad1.20x1.40mm_HandSolder, symbol Device:R_Small
- removed R2: 10, Resistor_SMD:R_0805_2012Metric_Pad1.20x1.40mm_HandSolder, symbol Device:R_Small
- removed TP906: ADC_DRDY, MEMS_Custom:TestPoint_Pad_D1.0mm, symbol Connector:TestPoint
- removed TP906: Anode_I, MEMS_Custom:TestPoint_Pad_D1.0mm, symbol Connector:TestPoint
- removed TP906: Grid_I, MEMS_Custom:TestPoint_Pad_D1.0mm, symbol Connector:TestPoint
- removed TP906: Cathode_I, MEMS_Custom:TestPoint_Pad_D1.0mm, symbol Connector:TestPoint
- removed TP906: SPI1_SCK, MEMS_Custom:TestPoint_Pad_D1.0mm, symbol Connector:TestPoint
- removed TP906: Cathode_V, MEMS_Custom:TestPoint_Pad_D1.0mm, symbol Connector:TestPoint
- removed TP907: ADC_RESET, MEMS_Custom:TestPoint_Pad_D1.0mm, symbol Connector:TestPoint
- removed TP907: SPI1_MISO, MEMS_Custom:TestPoint_Pad_D1.0mm, symbol Connector:TestPoint
- removed TP908: SPI1_MOSI, MEMS_Custom:TestPoint_Pad_D1.0mm, symbol Connector:TestPoint
- removed TP908: ADC_CS, MEMS_Custom:TestPoint_Pad_D1.0mm, symbol Connector:TestPoint
- removed TP909: SCL_INT, MEMS_Custom:TestPoint_Pad_D1.0mm, symbol Connector:TestPoint
- removed TP910: SDA_INT, MEMS_Custom:TestPoint_Pad_D1.0mm, symbol Connector:TestPoint
- removed U1: ADS131M04-WQFN, Package_DFN_QFN:WQFN-20-1EP_3x3mm_P0.4mm_EP1.7x1.7mm, symbol MEMS_IC:ADS131M04-WQFN
- removed X1: 8.192MHz, Oscillator:Oscillator_SMD_ECS_2520MV-xxx-xx-4Pin_2.5x2.0mm, symbol MEMS_IC:ECS-2520MVLC-081.92-CN-TR_oscillator_8.192MHZ
- added J1: Gauge Connector, Connector_IDC:IDC-Header_2x05_P2.54mm_Horizontal, symbol Connector:Conn_01x10_Pin
- added TP1: Grid_I, MEMS_Custom:TestPoint_Pad_D1.0mm, symbol Connector:TestPoint
- added TP2: Anode_I, MEMS_Custom:TestPoint_Pad_D1.0mm, symbol Connector:TestPoint
- added TP3: Cathode_I, MEMS_Custom:TestPoint_Pad_D1.0mm, symbol Connector:TestPoint
- added TP4: Cathode_V, MEMS_Custom:TestPoint_Pad_D1.0mm, symbol Connector:TestPoint
Connections:
- net GND: now also J1.10 (Pin_10), J1.9 (Pin_9)
- new net ADC/1: TP4.1
- new net ADC/2: TP3.1
- new net ADC/3: TP1.1
- new net ADC/4: TP2.1
- new net ANODE: J1.2 (Pin_2)
- new net CATHODE: J1.7 (Pin_7), J1.8 (Pin_8)
- new net GRID: J1.3 (Pin_3)
- no-connect marks 31 -> 4
Other:
- sheet EuroMeasure renamed MCU
- added sheet ADC (adc.kicad_sch)
- added sheet Anode Current Measurement (anode_ammeter.kicad_sch)
- added sheet Backplane connector (backplane_connector.kicad_sch)
- added sheet Grid Current Measurement (grid_current_measurement.kicad_sch)
- added sheet PSU (psu.kicad_sch)
- sheet Anode Supply ports: added +, -, 5V_IN; removed -25V_Anode_Supply, I_Monitor
- sheet Cathode Supply ports: added +, 15V_IN, I, V, {I2C}; removed Cathode_Supply, I_Monitor, SCL, SDA, U_Monitor
- sheet Grid Supply ports: added +, -, 5V_IN, ~{LOCKOUT}; removed 200V_Grid_Supply, I_Monitor
- sheet MCU: file ../EuroMeasure-Module/EuroMeasure.kicad_sch -> MCU.kicad_sch
- sheet MCU ports: added 3V3_IN, EXT{I2C}, INT{I2C}, {ADC}, {DEBUG}, {EM_MISC}; removed GP0, GP1, PA1, PA10, PA15, PA4, PA8, PA9, PB0, PB1, PB2, PB3, PB4, PB5, PC13, PC6, RDY, RGB_OUT, RX_DEBUG, SCL_EXT, SCL_INT, SDA_EXT, SDA_INT, SPI1_MISO, SPI1_MOSI, SPI1_SCK, SPI2_MISO, SPI2_MOSI, SPI2_SCK, SWCLK, SWDIO, TRG, TX_DEBUG, ~{LOCKOUT}
- note added: "A"
- note added: "ADC"
- note added: "Note: Only major power connections depicted in top level diagram"
- note added: "V"
- note removed: "-1.2V - 1.2V range"
- note removed: "MCU"
- note removed: "Overkill but already used elsewhere and supported by software"

Commit message: Everything clear. Gerbers generated
Parts:
- TP1: renamed from TP4; symbol Connector:TestPoint -> MEMS_Other:TP_1mm_via; now left out of the parts list
- TP2: renamed from TP3; symbol Connector:TestPoint -> MEMS_Other:TP_1mm_via; now left out of the parts list
- TP3: renamed from TP2; symbol Connector:TestPoint -> MEMS_Other:TP_1mm_via; now left out of the parts list
- TP4: renamed from TP1; symbol Connector:TestPoint -> MEMS_Other:TP_1mm_via; now left out of the parts list
Other:
- sheet Anode Current Measurement: file anode_ammeter.kicad_sch -> anode_current_measurement.kicad_sch
- note added: "Note: All digital interfaces use 3.3V logic levels"
Changed lines of the file:
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@@
     (effects (font (size 2 2)) (justify left bottom))
+  )
+  (text "Note: All digital interfaces\nuse 3.3V logic levels"
+    (at 91.44 177.8 0)
+    (effects (font (size 1.27 1.27)) (justify left bottom))
   )
   (text "A" (at 178.054 103.124 0)
@@
     (effects (font (size 1.27 1.27)) (justify left bottom))
   )
-  (label "~{LOCKOUT}" (at 76.2 105.41 0)
+  (label "~{LOCKOUT}" (at 76.2 105.41 0) (fields_autoplaced)
     (effects (font (size 1.27 1.27)) (justify left bottom))
   )
@@
     )
   )
-  (symbol (lib_id "Connector:TestPoint") (at 236.22 152.4 90) (mirror x) (unit 1)
-    (in_bom yes) (on_board yes) (dnp no)
-    (property "Reference" "TP2" (at 231.14 152.4 90)
+  (symbol (lib_id "MEMS_Other:TP_1mm_via") (at 236.22 152.4 90) (mirror x) (unit 1)
+    (in_bom no) (on_board yes) (dnp no)
+    (property "Reference" "TP3" (at 231.14 152.4 90)
       (effects (font (size 1.27 1.27)) (justify left))
     )
@@
       (effects (font (size 1.27 1.27)) (justify left))
     )
-    (property "Footprint" "MEMS_Custom:TestPoint_Pad_D1.0mm" (at 236.22 157.48 0)
-      (effects (font (size 1.27 1.27)) hide)
-    )
-    (property "Datasheet" "~" (at 236.22 157.48 0)
+    (property "Footprint" "MEMS_Custom:TestPoint_Pad_D1.0mm" (at 243.205 152.4 0)
+      (effects (font (size 1.27 1.27)) hide)
+    )
+    (property "Datasheet" "~" (at 247.015 152.4 0)
+      (effects (font (size 1.27 1.27)) hide)
+    )
+    (property "Sim.Enable" "0" (at 245.11 152.4 0)
+      (effects (font (size 1.27 1.27)) hide)
+    )
+    (pin "1")
+    (instances
+      (project "EuroMeasure-IonGaugeController"
+        (path "/9c84a828-ebcc-4f88-b5cc-11be4f5044ad"
+          (reference "TP3") (unit 1)
+        )
+      )
+    )
+  )
+  (symbol (lib_id "MEMS_Other:TP_1mm_via") (at 236.22 139.7 90) (mirror x) (unit 1)
+    (in_bom no) (on_board yes) (dnp no)
+    (property "Reference" "TP2" (at 231.14 139.7 90)
+      (effects (font (size 1.27 1.27)) (justify left))
+    )
+    (property "Value" "Cathode_I" (at 224.79 139.7 90)
+      (effects (font (size 1.27 1.27)) (justify left))
+    )
+    (property "Footprint" "MEMS_Custom:TestPoint_Pad_D1.0mm" (at 243.205 139.7 0)
+      (effects (font (size 1.27 1.27)) hide)
+    )
+    (property "Datasheet" "~" (at 247.015 139.7 0)
+      (effects (font (size 1.27 1.27)) hide)
+    )
+    (property "Sim.Enable" "0" (at 245.11 139.7 0)
       (effects (font (size 1.27 1.27)) hide)
     )
@@
         (path "/9c84a828-ebcc-4f88-b5cc-11be4f5044ad"
           (reference "TP2") (unit 1)
-        )
-      )
-    )
-  )
-  (symbol (lib_id "Connector:TestPoint") (at 236.22 139.7 90) (mirror x) (unit 1)
-    (in_bom yes) (on_board yes) (dnp no)
-    (property "Reference" "TP3" (at 231.14 139.7 90)
-      (effects (font (size 1.27 1.27)) (justify left))
-    )
-    (property "Value" "Cathode_I" (at 224.79 139.7 90)
-      (effects (font (size 1.27 1.27)) (justify left))
-    )
-    (property "Footprint" "MEMS_Custom:TestPoint_Pad_D1.0mm" (at 236.22 144.78 0)
-      (effects (font (size 1.27 1.27)) hide)
-    )
-    (property "Datasheet" "~" (at 236.22 144.78 0)
-      (effects (font (size 1.27 1.27)) hide)
-    )
-    (pin "1")
-    (instances
-      (project "EuroMeasure-IonGaugeController"
-        (path "/9c84a828-ebcc-4f88-b5cc-11be4f5044ad"
-          (reference "TP3") (unit 1)
         )
       )
@@
   (symbol (lib_id "power:+3.3V") (at 115.57 39.37 0) (unit 1)
     (in_bom yes) (on_board yes) (dnp no)
-    (property "Reference" "#PWR011" (at 115.57 43.18 0)
+    (property "Reference" "#PWR04" (at 115.57 43.18 0)
       (effects (font (size 1.27 1.27)) hide)
     )
@@
       (project "EuroMeasure-IonGaugeController"
         (path "/9c84a828-ebcc-4f88-b5cc-11be4f5044ad"
-          (reference "#PWR011") (unit 1)
+          (reference "#PWR04") (unit 1)
         )
       )
@@
   (symbol (lib_id "power:+15V") (at 59.69 72.39 0) (unit 1)
     (in_bom yes) (on_board yes) (dnp no) (fields_autoplaced)
-    (property "Reference" "#PWR04" (at 59.69 76.2 0)
+    (property "Reference" "#PWR02" (at 59.69 76.2 0)
       (effects (font (size 1.27 1.27)) hide)
     )
@@
       (project "EuroMeasure-IonGaugeController"
         (path "/9c84a828-ebcc-4f88-b5cc-11be4f5044ad"
-          (reference "#PWR04") (unit 1)
+          (reference "#PWR02") (unit 1)
         )
       )
@@
   (symbol (lib_id "power:-15V") (at 64.77 72.39 0) (unit 1)
     (in_bom yes) (on_board yes) (dnp no) (fields_autoplaced)
-    (property "Reference" "#PWR08" (at 64.77 69.85 0)
+    (property "Reference" "#PWR03" (at 64.77 69.85 0)
       (effects (font (size 1.27 1.27)) hide)
     )
@@
       (project "EuroMeasure-IonGaugeController"
         (path "/9c84a828-ebcc-4f88-b5cc-11be4f5044ad"
-          (reference "#PWR08") (unit 1)
-        )
-      )
-    )
-  )
-  (symbol (lib_id "Connector:TestPoint") (at 237.49 146.05 90) (mirror x) (unit 1)
-    (in_bom yes) (on_board yes) (dnp no)
-    (property "Reference" "TP1" (at 232.41 146.05 90)
+          (reference "#PWR03") (unit 1)
+        )
+      )
+    )
+  )
+  (symbol (lib_id "MEMS_Other:TP_1mm_via") (at 237.49 146.05 90) (mirror x) (unit 1)
+    (in_bom no) (on_board yes) (dnp no)
+    (property "Reference" "TP4" (at 232.41 146.05 90)
       (effects (font (size 1.27 1.27)) (justify left))
     )
@@
       (effects (font (size 1.27 1.27)) (justify left))
     )
-    (property "Footprint" "MEMS_Custom:TestPoint_Pad_D1.0mm" (at 237.49 151.13 0)
-      (effects (font (size 1.27 1.27)) hide)
-    )
-    (property "Datasheet" "~" (at 237.49 151.13 0)
+    (property "Footprint" "MEMS_Custom:TestPoint_Pad_D1.0mm" (at 244.475 146.05 0)
+      (effects (font (size 1.27 1.27)) hide)
+    )
+    (property "Datasheet" "~" (at 248.285 146.05 0)
+      (effects (font (size 1.27 1.27)) hide)
+    )
+    (property "Sim.Enable" "0" (at 246.38 146.05 0)
+      (effects (font (size 1.27 1.27)) hide)
+    )
+    (pin "1")
+    (instances
+      (project "EuroMeasure-IonGaugeController"
+        (path "/9c84a828-ebcc-4f88-b5cc-11be4f5044ad"
+          (reference "TP4") (unit 1)
+        )
+      )
+    )
+  )
+  (symbol (lib_id "MEMS_Other:TP_1mm_via") (at 236.22 133.35 90) (mirror x) (unit 1)
+    (in_bom no) (on_board yes) (dnp no)
+    (property "Reference" "TP1" (at 231.14 133.35 90)
+      (effects (font (size 1.27 1.27)) (justify left))
+    )
+    (property "Value" "Cathode_V" (at 224.79 133.35 90)
+      (effects (font (size 1.27 1.27)) (justify left))
+    )
+    (property "Footprint" "MEMS_Custom:TestPoint_Pad_D1.0mm" (at 243.205 133.35 0)
+      (effects (font (size 1.27 1.27)) hide)
+    )
+    (property "Datasheet" "~" (at 247.015 133.35 0)
+      (effects (font (size 1.27 1.27)) hide)
+    )
+    (property "Sim.Enable" "0" (at 245.11 133.35 0)
       (effects (font (size 1.27 1.27)) hide)
     )
@@
         (path "/9c84a828-ebcc-4f88-b5cc-11be4f5044ad"
           (reference "TP1") (unit 1)
-        )
-      )
-    )
-  )
-  (symbol (lib_id "Connector:TestPoint") (at 236.22 133.35 90) (mirror x) (unit 1)
-    (in_bom yes) (on_board yes) (dnp no)
-    (property "Reference" "TP4" (at 231.14 133.35 90)
-      (effects (font (size 1.27 1.27)) (justify left))
-    )
-    (property "Value" "Cathode_V" (at 224.79 133.35 90)
-      (effects (font (size 1.27 1.27)) (justify left))
-    )
-    (property "Footprint" "MEMS_Custom:TestPoint_Pad_D1.0mm" (at 236.22 138.43 0)
-      (effects (font (size 1.27 1.27)) hide)
-    )
-    (property "Datasheet" "~" (at 236.22 138.43 0)
-      (effects (font (size 1.27 1.27)) hide)
-    )
-    (pin "1")
-    (instances
-      (project "EuroMeasure-IonGaugeController"
-        (path "/9c84a828-ebcc-4f88-b5cc-11be4f5044ad"
-          (reference "TP4") (unit 1)
         )
       )
@@
   (symbol (lib_id "power:GND") (at 236.22 69.85 0) (unit 1)
     (in_bom yes) (on_board yes) (dnp no) (fields_autoplaced)
-    (property "Reference" "#PWR018" (at 236.22 76.2 0)
+    (property "Reference" "#PWR05" (at 236.22 76.2 0)
       (effects (font (size 1.27 1.27)) hide)
     )
@@
       (project "EuroMeasure-IonGaugeController"
         (path "/9c84a828-ebcc-4f88-b5cc-11be4f5044ad"
-          (reference "#PWR018") (unit 1)
+          (reference "#PWR05") (unit 1)
         )
       )
@@
       (effects (font (size 2 2)) (justify left bottom))
     )
-    (property "Sheetfile" "anode_ammeter.kicad_sch" (at 173.99 34.8746 0)
-      (effects (font (size 1.27 1.27)) (justify left top) hide)
-    )
+    (property "Sheetfile" "anode_current_measurement.kicad_sch" (at 173.99 34.8746 0)
+      (effects (font (size 1.27 1.27)) (justify left top) hide)
+    )
