File: EuroMeasure-IonGaugeController.kicad_sch (KiCad schematic)
At the start: 5 parts, among them J1 Gauge Connector

Commit message: Exported auxiliary files
Parts:
- J1: MPN (none) -> 61201021721; Mouser (none) -> 710-61201021721
Other:
- sheet ADC: file adc.kicad_sch -> sch/adc.kicad_sch
- sheet Anode Current Measurement: file anode_current_measurement.kicad_sch -> sch/anode_current_measurement.kicad_sch
- sheet Anode Supply: file anode_supply.kicad_sch -> sch/anode_supply.kicad_sch
- sheet Backplane connector: file backplane_connector.kicad_sch -> sch/backplane_connector.kicad_sch
- sheet Cathode Supply: file cathode_supply.kicad_sch -> sch/cathode_supply.kicad_sch
- sheet Grid Current Measurement: file grid_current_measurement.kicad_sch -> sch/grid_current_measurement.kicad_sch
- sheet Grid Supply: file grid_supply.kicad_sch -> sch/grid_supply.kicad_sch
- sheet MCU: file MCU.kicad_sch -> sch/MCU.kicad_sch
- sheet PSU: file psu.kicad_sch -> sch/psu.kicad_sch
Changed lines of the file:
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@@
+      (effects (font (size 1.27 1.27)) hide)
+    )
+    (property "MPN" "61201021721" (at 245.11 55.88 0)
+      (effects (font (size 1.27 1.27)) hide)
+    )
+    (property "Mouser" "710-61201021721" (at 245.11 55.88 0)
       (effects (font (size 1.27 1.27)) hide)
     )
@@
       (effects (font (size 3 3)) (justify left bottom))
     )
-    (property "Sheetfile" "cathode_supply.kicad_sch" (at 152.4 121.2346 0)
+    (property "Sheetfile" "sch/cathode_supply.kicad_sch" (at 152.4 121.2346 0)
       (effects (font (size 1.27 1.27)) (justify left top) hide)
     )
@@
       (effects (font (size 3 3)) (justify left bottom))
     )
-    (property "Sheetfile" "grid_supply.kicad_sch" (at 133.35 69.1646 0)
+    (property "Sheetfile" "sch/grid_supply.kicad_sch" (at 133.35 69.1646 0)
       (effects (font (size 1.27 1.27)) (justify left top) hide)
     )
@@
       (effects (font (size 3 3)) (justify left bottom))
     )
-    (property "Sheetfile" "anode_supply.kicad_sch" (at 133.35 45.0346 0)
+    (property "Sheetfile" "sch/anode_supply.kicad_sch" (at 133.35 45.0346 0)
       (effects (font (size 1.27 1.27)) (justify left top) hide)
     )
@@
       (effects (font (size 2 2)) (justify left bottom))
     )
-    (property "Sheetfile" "grid_current_measurement.kicad_sch" (at 173.99 85.6746 0)
+    (property "Sheetfile" "sch/grid_current_measurement.kicad_sch" (at 173.99 85.6746 0)
       (effects (font (size 1.27 1.27)) (justify left top) hide)
     )
@@
       (effects (font (size 3 3)) (justify left bottom))
     )
-    (property "Sheetfile" "adc.kicad_sch" (at 240.03 159.3346 0)
+    (property "Sheetfile" "sch/adc.kicad_sch" (at 240.03 159.3346 0)
       (effects (font (size 1.27 1.27)) (justify left top) hide)
     )
@@
       (effects (font (size 2 2)) (justify left bottom))
     )
-    (property "Sheetfile" "anode_current_measurement.kicad_sch" (at 173.99 34.8746 0)
+    (property "Sheetfile" "sch/anode_current_measurement.kicad_sch" (at 173.99 34.8746 0)
       (effects (font (size 1.27 1.27)) (justify left top) hide)
     )
@@
       (effects (font (size 3 3)) (justify left bottom))
     )
-    (property "Sheetfile" "backplane_connector.kicad_sch" (at 27.94 99.6446 0)
+    (property "Sheetfile" "sch/backplane_connector.kicad_sch" (at 27.94 99.6446 0)
       (effects (font (size 1.27 1.27)) (justify left top) hide)
     )
@@
       (effects (font (size 3 3)) (justify left bottom))
     )
-    (property "Sheetfile" "MCU.kicad_sch" (at 87.63 173.3046 0)
+    (property "Sheetfile" "sch/MCU.kicad_sch" (at 87.63 173.3046 0)
       (effects (font (size 1.27 1.27)) (justify left top) hide)
     )
@@
       (effects (font (size 3 3)) (justify left bottom))
     )
-    (property "Sheetfile" "psu.kicad_sch" (at 81.28 56.4646 0)
-      (effects (font (size 1.27 1.27)) (justify left top) hide)
-    )
+    (property "Sheetfile" "sch/psu.kicad_sch" (at 81.28 56.4646 0)
+      (effects (font (size 1.27 1.27)) (justify left top) hide)
+    )
